Commit message: working with real meshes

File: gbeam_model/urdf/gbeam_link.urdf (robot description, URDF)
Before this commit: robot gbeam_link, 1 links, 0 joints
Links:
- link gbeam_link: geometry visual mesh filename=package://gbeam_model/meshes/gbeam_link_50k.dae

File: gbeam_sim/gbeam.world.xacro (robot description, xacro)
@@ -15,4 +15,6 @@
         <frameId>hog</frameId>
         <linkName>hog</linkName>
+        <kl>10000</kl>
+        <ka>200</ka>
       </plugin>
       <link name ='hog'>
@@ -29,4 +31,12 @@
           </geometry>
         </visual>
+        <inertial>
+          <mass>0.3</mass>
+          <inertia>
+            <ixx>0.001</ixx><ixy>0</ixy>    <ixz>0</ixz>
+            <iyy>0.001</iyy><iyz>0</iyz>
+            <izz>0.001</izz>
+          </inertia>
+        </inertial>
       </link>
     </model>

File: gbeam_sim/gbeam_soup.sdf.xacro (robot description, xacro)
@@ -16,14 +16,18 @@
       <collision name='collision'>
         <geometry>
-          <box>
-            <size>0.05 0.3 0.05</size>
-          </box>
+          <mesh><uri>file://$(find gbeam_model)/meshes/gbeam_link_50k.dae</uri></mesh>
         </geometry>
+        <surface>
+          <friction>
+            <ode>
+              <mu>1.0</mu>
+              <mu2>0.7</mu2>
+            </ode>
+          </friction>
+        </surface>
       </collision>
       <visual name='visual'>
         <geometry>
-          <box>
-            <size>0.05 0.3 0.05</size>
-          </box>
+          <mesh><uri>file://$(find gbeam_model)/meshes/gbeam_link_50k.dae</uri></mesh>
         </geometry>
       </visual>
@@ -44,14 +48,18 @@
       <collision name='collision'>
         <geometry>
-          <box>
-            <size>0.05 0.05 0.05</size>
-          </box>
+          <mesh><uri>file://$(find gbeam_model)/meshes/gbeam_node_25k.dae</uri></mesh>
         </geometry>
+        <surface>
+          <friction>
+            <ode>
+              <mu>0.5</mu>
+              <mu2>0.5</mu2>
+            </ode>
+          </friction>
+        </surface>
       </collision>
       <visual name='visual'>
         <geometry>
-          <box>
-            <size>0.05 0.05 0.05</size>
-          </box>
+          <mesh><uri>file://$(find gbeam_model)/meshes/gbeam_node_25k.dae</uri></mesh>
         </geometry>
       </visual>
@@ -60,6 +68,5 @@
   <model name="gbeam_soup">
     <plugin name="assembly_soup" filename="libassembly_soup_plugin.so">
-      <trans_mate_err>0.01</trans_mate_err>
-      <rot_mate_err>0.1</rot_mate_err>
+      <!-- Frame that poses are broadcasted in -->
       <tf_world_frame>world</tf_world_frame>
       <!-- Mate Models -->
@@ -71,4 +78,12 @@
           <rot>1 1 4</rot>
         </symmetry>
+        <attach_threshold>
+          <linear>0.01</linear>
+          <angular>0.1</angular>
+        </attach_threshold>
+        <detach_threshold>
+          <linear>0.015</linear>
+          <angular>0.2</angular>
+        </detach_threshold>
         <joint type="prismatic" name="gbeam">
           <pose>0 0.025 0 0 ${pi/2} 0</pose>
@@ -95,37 +110,37 @@
       <atom_model type="gbeam_link">
         <mate_point type="gbeam" gender="male">
-          <pose>0 0.15 0 ${pi/2} 0 ${pi}</pose>
+          <pose>0 0.125 0 ${pi/2} ${pi/4} ${pi}</pose>
         </mate_point>
-        <!--<mate_point type="gbeam" gender="male">-->
-          <!--<pose>0 -0.100 0 -${pi/2.0} 0 0</pose>-->
-        <!--</mate_point>-->
+        <mate_point type="gbeam" gender="male">
+          <pose>0 -0.125 0 ${pi/2} ${pi/4} 0</pose>
+        </mate_point>
       </atom_model>
       <atom_model type="gbeam_node">
-        <!--<mate_point type="gbeam" gender="female">-->
-          <!--<pose>0 0.025 0 ${pi/2} 0 0</pose>-->
-        <!--</mate_point>-->
+        <mate_point type="gbeam" gender="female">
+          <pose>0 0.025 0 ${pi/2} 0 0</pose>
+        </mate_point>
         <mate_point type="gbeam" gender="female">
           <pose>0 -0.025 0 ${pi/2} 0 ${pi}</pose>
         </mate_point>
-        <!--<mate_point type="gbeam" gender="female">-->
-          <!--<pose>0 0.05 0 -${pi/2.0} 0 0</pose>-->
-        <!--</mate_point>-->
-        <!--<mate_point type="gbeam" gender="female">-->
-          <!--<pose>0 -0.05 0 ${pi/2.0} 0 0</pose>-->
-        <!--</mate_point>-->
-        <!--<mate_point type="gbeam" gender="female">-->
-          <!--<pose>0.05 0 0 0 ${pi/2.0} 0</pose>-->
-        <!--</mate_point>-->
-        <!--<mate_point type="gbeam" gender="female">-->
-          <!--<pose>-0.05 0 0 0 -${pi/2.0} 0</pose>-->
-        <!--</mate_point>-->
+        <mate_point type="gbeam" gender="female">
+          <pose>0 0 0.025 ${pi} 0 0</pose>
+        </mate_point>
+        <mate_point type="gbeam" gender="female">
+          <pose>0 0 -0.025 0 0 0</pose>
+        </mate_point>
+        <mate_point type="gbeam" gender="female">
+          <pose>0.025 0 0 0 -${pi/2.0} 0</pose>
+        </mate_point>
+        <mate_point type="gbeam" gender="female">
+          <pose>-0.025 0 0 0 ${pi/2.0} 0</pose>
+        </mate_point>
       </atom_model>
     </plugin>
-    <xacro:gbeam_node suffix="_1" pose="0 0.3 0 0 0 0"/>
+    <xacro:gbeam_node suffix="_1" pose="0 0.3 0.2 0 0 0"/>
     <!--<xacro:gbeam_node suffix="_2" pose="0 0 0.1 0 0 0"/>-->
     <!--<xacro:gbeam_node suffix="_3" pose="0 0 0.2 0 0 0"/>-->
     <!--<xacro:gbeam_node suffix="_4" pose="0 0 0.3 0 0 0"/>-->
     <!--<xacro:gbeam_node suffix="_5" pose="0 0 0.4 0 0 0"/>-->
-    <xacro:gbeam_link suffix="_1" pose="0 0 0 0 0 0"/>
+    <xacro:gbeam_link suffix="_1" pose="0 0 0.2 0 0 0"/>
     <!--<xacro:gbeam_link suffix="_2" pose="0 0.1 0.1 0 0 0"/>-->
     <!--<xacro:gbeam_link suffix="_3" pose="0 0.1 0.2 0 0 0"/>-->
