Commit message: getting closer to working assembly plugin

File: gbeam_sim/gbeam.world.xacro (robot description, xacro)
@@ -10,155 +10,156 @@
       <uri>model://ground_plane</uri>
     </include>
-    <model name ='hog'>
-      <plugin name='hand_of_god' filename="libgazebo_ros_hand_of_god.so">
-        <frameId>hydra_right_grab</frameId>
-        <linkName>hog</linkName>
-      </plugin>
-      <link name ='hog'>
+    <xacro:if value="0">
+      <model name ='hog'>
+        <plugin name='hand_of_god' filename="libgazebo_ros_hand_of_god.so">
+          <frameId>hydra_right_grab</frameId>
+          <linkName>hog</linkName>
+        </plugin>
+        <link name ='hog'>
+          <self_collide>0</self_collide>
+          <pose>0 0 0 0 0 0</pose>
+          <collision name ='collision'>
+            <geometry>
+              <sphere><radius>0.5</radius></sphere>
+            </geometry>
+          </collision>
+          <visual name ='visual'>
+            <geometry>
+              <sphere><radius>0.5</radius></sphere>
+            </geometry>
+          </visual>
+        </link>
+      </model>
+      <xacro:macro name="gbeam_node">
         <self_collide>0</self_collide>
-        <pose>0 0 0 0 0 0</pose>
         <collision name ='collision'>
           <geometry>
-            <sphere><radius>0.5</radius></sphere>
+            <box><size>1 1 1</size></box>
           </geometry>
         </collision>
         <visual name ='visual'>
           <geometry>
-            <sphere><radius>0.5</radius></sphere>
+            <box><size>1 1 1</size></box>
           </geometry>
         </visual>
-      </link>
-    </model>
-    <xacro:macro name="gbeam_node">
-      <self_collide>0</self_collide>
-      <collision name ='collision'>
-        <geometry>
-          <box><size>1 1 1</size></box>
-        </geometry>
-      </collision>
-      <visual name ='visual'>
-        <geometry>
-          <box><size>1 1 1</size></box>
-        </geometry>
-      </visual>
-    </xacro:macro>
-    <xacro:macro name="gbeam_link">
-      <self_collide>0</self_collide>
-      <collision name ='collision'>
-        <geometry>
-          <box><size>0.2 4 0.2</size></box>
-        </geometry>
-      </collision>
-      <visual name ='visual'>
-        <geometry>
-          <box><size>0.2 4 0.2</size></box>
-        </geometry>
-      </visual>
-    </xacro:macro>
-    <xacro:macro name="gbeam_mate">
-      <axis>
-        <xyz>1 0 0</xyz>
-        <limit><lower>0</lower><upper>0</upper></limit>
-      </axis>
-      <physics>
-        <ode>
-          <cfm_damping>1</cfm_damping>
-          <cfm>0.1</cfm>
-          <erp>0.1</erp>
-          <limit>
+      </xacro:macro>
+      <xacro:macro name="gbeam_link">
+        <self_collide>0</self_collide>
+        <collision name ='collision'>
+          <geometry>
+            <box><size>0.2 4 0.2</size></box>
+          </geometry>
+        </collision>
+        <visual name ='visual'>
+          <geometry>
+            <box><size>0.2 4 0.2</size></box>
+          </geometry>
+        </visual>
+      </xacro:macro>
+      <xacro:macro name="gbeam_mate">
+        <axis>
+          <xyz>1 0 0</xyz>
+          <limit><lower>0</lower><upper>0</upper></limit>
+        </axis>
+        <physics>
+          <ode>
+            <cfm_damping>1</cfm_damping>
             <cfm>0.1</cfm>
             <erp>0.1</erp>
-          </limit>
-        </ode>
-      </physics>
-    </xacro:macro>
-    <xacro:property name="gbeam_mate_joint_type" value="revolute"/>
-    <xacro:property name="pi" value="3.14159265"/>
-    <model name ='assembly'>
-      <pose>1 2 10 0 0.2 0</pose>
-      <link name ='node1'>
-        <pose>0 0 .5 0 0 0</pose>
-        <xacro:gbeam_node/>
-      </link>
-      <joint type="${gbeam_mate_joint_type}" name='n1l12'>
-        <pose>0 -2 0 0 0 0</pose>
-        <parent>node1</parent>
-        <child>link12</child>
-        <xacro:gbeam_mate/>
-      </joint>
-      <link name ='link12'>
-        <self_collide>1</self_collide>
-        <pose>0 2.5 .5 0 0 0</pose>
-        <xacro:gbeam_link/>
-      </link>
-      <joint type="${gbeam_mate_joint_type}" name='l12n2'>
-        <pose>0 2 0 0 0 0</pose>
-        <parent>node2</parent>
-        <child>link12</child>
-        <xacro:gbeam_mate/>
-      </joint>
-      <link name ='node2'>
-        <pose>0 5 0.5 0 0 0</pose>
-        <xacro:gbeam_node/>
-      </link>
-      <joint type="${gbeam_mate_joint_type}" name='n2l23'>
-        <pose>0 -2 0 0 0 0</pose>
-        <parent>node2</parent>
-        <child>link23</child>
-        <xacro:gbeam_mate/>
-      </joint>
-      <link name ='link23'>
-        <pose>0 5 3 ${pi/2.0} 0 0</pose>
-        <xacro:gbeam_link/>
-      </link>
-      <joint type="${gbeam_mate_joint_type}" name='l23n3'>
-        <pose>0 2 0 0 0 0</pose>
-        <parent>node3</parent>
-        <child>link23</child>
-        <xacro:gbeam_mate/>
-      </joint>
-      <link name ='node3'>
-        <pose>0 5 5.5 0 0 0</pose>
-        <xacro:gbeam_node/>
-      </link>
-      <joint type="${gbeam_mate_joint_type}" name='n3l34'>
-        <pose>0 2 0 0 0 0</pose>
-        <parent>node3</parent>
-        <child>link34</child>
-        <xacro:gbeam_mate/>
-      </joint>
-      <link name ='link34'>
-        <pose>0 2.5 5.5 0 0 0</pose>
-        <xacro:gbeam_link/>
-      </link>
-      <joint type="${gbeam_mate_joint_type}" name='l34n4'>
-        <pose>0 -2 0 0 0 0</pose>
-        <parent>node4</parent>
-        <child>link34</child>
-        <xacro:gbeam_mate/>
-      </joint>
-      <link name ='node4'>
-        <pose>0 0 5.5 0 0 0</pose>
-        <xacro:gbeam_node/>
-      </link>
-      <joint type="${gbeam_mate_joint_type}" name='n4l41'>
-        <pose>0 2 0 0 0 0</pose>
-        <parent>node4</parent>
-        <child>link41</child>
-        <xacro:gbeam_mate/>
-      </joint>
-      <link name ='link41'>
-        <pose>0 0 3 ${pi/2.0} 0 0</pose>
-        <xacro:gbeam_link/>
-      </link>
-      <joint type="${gbeam_mate_joint_type}" name='l41n1'>
-        <pose>0 -2 0 0 0 0</pose>
-        <parent>node1</parent>
-        <child>link41</child>
-        <xacro:gbeam_mate/>
-      </joint>
-      <xacro:if value="0">
-      </xacro:if>
-    </model>
+            <limit>
+              <cfm>0.1</cfm>
+              <erp>0.1</erp>
+            </limit>
+          </ode>
+        </physics>
+      </xacro:macro>
+      <xacro:property name="gbeam_mate_joint_type" value="revolute"/>
+      <xacro:property name="pi" value="3.14159265"/>
+      <model name ='assembly'>
+        <pose>1 2 10 0 0.2 0</pose>
+        <link name ='node1'>
+          <pose>0 0 .5 0 0 0</pose>
+          <xacro:gbeam_node/>
+        </link>
+        <joint type="${gbeam_mate_joint_type}" name='n1l12'>
+          <pose>0 -2 0 0 0 0</pose>
+          <parent>node1</parent>
+          <child>link12</child>
+          <xacro:gbeam_mate/>
+        </joint>
+        <link name ='link12'>
+          <self_collide>1</self_collide>
+          <pose>0 2.5 .5 0 0 0</pose>
+          <xacro:gbeam_link/>
+        </link>
+        <joint type="${gbeam_mate_joint_type}" name='l12n2'>
+          <pose>0 2 0 0 0 0</pose>
+          <parent>node2</parent>
+          <child>link12</child>
+          <xacro:gbeam_mate/>
+        </joint>
+        <link name ='node2'>
+          <pose>0 5 0.5 0 0 0</pose>
+          <xacro:gbeam_node/>
+        </link>
+        <joint type="${gbeam_mate_joint_type}" name='n2l23'>
+          <pose>0 -2 0 0 0 0</pose>
+          <parent>node2</parent>
+          <child>link23</child>
+          <xacro:gbeam_mate/>
+        </joint>
+        <link name ='link23'>
+          <pose>0 5 3 ${pi/2.0} 0 0</pose>
+          <xacro:gbeam_link/>
+        </link>
+        <joint type="${gbeam_mate_joint_type}" name='l23n3'>
+          <pose>0 2 0 0 0 0</pose>
+          <parent>node3</parent>
+          <child>link23</child>
+          <xacro:gbeam_mate/>
+        </joint>
+        <link name ='node3'>
+          <pose>0 5 5.5 0 0 0</pose>
+          <xacro:gbeam_node/>
+        </link>
+        <joint type="${gbeam_mate_joint_type}" name='n3l34'>
+          <pose>0 2 0 0 0 0</pose>
+          <parent>node3</parent>
+          <child>link34</child>
+          <xacro:gbeam_mate/>
+        </joint>
+        <link name ='link34'>
+          <pose>0 2.5 5.5 0 0 0</pose>
+          <xacro:gbeam_link/>
+        </link>
+        <joint type="${gbeam_mate_joint_type}" name='l34n4'>
+          <pose>0 -2 0 0 0 0</pose>
+          <parent>node4</parent>
+          <child>link34</child>
+          <xacro:gbeam_mate/>
+        </joint>
+        <link name ='node4'>
+          <pose>0 0 5.5 0 0 0</pose>
+          <xacro:gbeam_node/>
+        </link>
+        <joint type="${gbeam_mate_joint_type}" name='n4l41'>
+          <pose>0 2 0 0 0 0</pose>
+          <parent>node4</parent>
+          <child>link41</child>
+          <xacro:gbeam_mate/>
+        </joint>
+        <link name ='link41'>
+          <pose>0 0 3 ${pi/2.0} 0 0</pose>
+          <xacro:gbeam_link/>
+        </link>
+        <joint type="${gbeam_mate_joint_type}" name='l41n1'>
+          <pose>0 -2 0 0 0 0</pose>
+          <parent>node1</parent>
+          <child>link41</child>
+          <xacro:gbeam_mate/>
+        </joint>
+      </model>
+    </xacro:if>
+    <xacro:include filename="$(find gbeam_sim)/gbeam_soup.sdf.xacro"/>
   </world>
 </sdf>

File: gbeam_sim/gbeam_soup.sdf.xacro (robot description, xacro)
@@ -1,9 +1,9 @@
 <?xml version='1.0'?>
-<sdf version='1.4'>
+<sdf version="1.4" xmlns:xacro="http://www.ros.org/wiki/xacro" >
   <xacro:property name="pi" value="3.14159265"/>
   <model name="gbeam_soup">
-    <plugin name="assembly_soup" filename="libassembly_soup.so">
-      <!-- Mate Templates -->
-      <mate_template type="gbeam">
+    <plugin name="assembly_soup" filename="libassembly_soup_plugin.so">
+      <!-- Mate Models -->
+      <mate_model type="gbeam">
         <!-- planar shear-supporting magnetic mate
              mating surface is along positive z-axis
@@ -32,8 +32,10 @@
           </physics>
         </joint>
-      </mate_template>
-      <!-- Atom Templates -->
-      <atom_template type="gbeam_link">
+      </mate_model>
+      <!-- Atom Models -->
+      <atom_model type="gbeam_link">
         <link name="gbeam_link">
+          <pose>0 0 0 0 0 0</pose>
+          <self_collide>0</self_collide>
           <inertial>
             <mass>0.3</mass>
@@ -59,13 +61,15 @@
           </visual>
         </link>
-        <mate type="gbeam" gender="male">
+        <mate_point type="gbeam" gender="male">
           <pose>0 0.100 0 ${pi/2.0} 0 0</pose>
-        </mate>
-        <mate type="gbeam" gender="male">
+        </mate_point>
+        <mate_point type="gbeam" gender="male">
           <pose>0 -0.100 0 -${pi/2.0} 0 0</pose>
-        </mate>
-      </atom_template>
-      <atom_template type="gbeam_node">
+        </mate_point>
+      </atom_model>
+      <atom_model type="gbeam_node">
         <link name="gbeam_node">
+          <pose>0 0 0 0 0 0</pose>
+          <self_collide>0</self_collide>
           <inertial>
             <mass>0.2</mass>
@@ -91,23 +95,23 @@
           </visual>
         </link>
-        <mate type="gbeam" gender="female">
+        <mate_point type="gbeam" gender="female">
           <pose>0 0 0.5 0 0 0</pose>
-        </mate>
-        <mate type="gbeam" gender="female">
+        </mate_point>
+        <mate_point type="gbeam" gender="female">
           <pose>0 0 -0.05 0 0 ${pi}</pose>
-        </mate>
-        <mate type="gbeam" gender="female">
+        </mate_point>
+        <mate_point type="gbeam" gender="female">
           <pose>0 0.05 0 -${pi/2.0} 0 0</pose>
-        </mate>
-        <mate type="gbeam" gender="female">
+        </mate_point>
+        <mate_point type="gbeam" gender="female">
           <pose>0 -0.05 0 ${pi/2.0} 0 0</pose>
-        </mate>
-        <mate type="gbeam" gender="female">
+        </mate_point>
+        <mate_point type="gbeam" gender="female">
           <pose>0.05 0 0 0 ${pi/2.0} 0</pose>
-        </mate>
-        <mate type="gbeam" gender="female">
+        </mate_point>
+        <mate_point type="gbeam" gender="female">
           <pose>-0.05 0 0 0 -${pi/2.0} 0</pose>
-        </mate>
-      </atom_template>
+        </mate_point>
+      </atom_model>
       <assembly>
         <atom type="gbeam_node">

Commit message: added run deps; added sdf tags to set rotational and translational error

File: gbeam_sim/gbeam.world.xacro (robot description, xacro)
@@ -10,5 +10,5 @@
       <uri>model://ground_plane</uri>
     </include>
-    <xacro:if value="0">
+    <xacro:if value="1">
       <model name ='hog'>
         <plugin name='hand_of_god' filename="libgazebo_ros_hand_of_god.so">
@@ -18,147 +18,18 @@
         <link name ='hog'>
           <self_collide>0</self_collide>
-          <pose>0 0 0 0 0 0</pose>
+          <pose>0 0 1 0 0 0</pose>
           <collision name ='collision'>
             <geometry>
-              <sphere><radius>0.5</radius></sphere>
+              <sphere><radius>0.025</radius></sphere>
             </geometry>
           </collision>
           <visual name ='visual'>
             <geometry>
-              <sphere><radius>0.5</radius></sphere>
+              <sphere><radius>0.025</radius></sphere>
             </geometry>
           </visual>
         </link>
       </model>
-      <xacro:macro name="gbeam_node">
-        <self_collide>0</self_collide>
-        <collision name ='collision'>
-          <geometry>
-            <box><size>1 1 1</size></box>
-          </geometry>
-        </collision>
-        <visual name ='visual'>
-          <geometry>
-            <box><size>1 1 1</size></box>
-          </geometry>
-        </visual>
-      </xacro:macro>
-      <xacro:macro name="gbeam_link">
-        <self_collide>0</self_collide>
-        <collision name ='collision'>
-          <geometry>
-            <box><size>0.2 4 0.2</size></box>
-          </geometry>
-        </collision>
-        <visual name ='visual'>
-          <geometry>
-            <box><size>0.2 4 0.2</size></box>
-          </geometry>
-        </visual>
-      </xacro:macro>
-      <xacro:macro name="gbeam_mate">
-        <axis>
-          <xyz>1 0 0</xyz>
-          <limit><lower>0</lower><upper>0</upper></limit>
-        </axis>
-        <physics>
-          <ode>
-            <cfm_damping>1</cfm_damping>
-            <cfm>0.1</cfm>
-            <erp>0.1</erp>
-            <limit>
-              <cfm>0.1</cfm>
-              <erp>0.1</erp>
-            </limit>
-          </ode>
-        </physics>
-      </xacro:macro>
-      <xacro:property name="gbeam_mate_joint_type" value="revolute"/>
-      <xacro:property name="pi" value="3.14159265"/>
-      <model name ='assembly'>
-        <pose>1 2 10 0 0.2 0</pose>
-        <link name ='node1'>
-          <pose>0 0 .5 0 0 0</pose>
-          <xacro:gbeam_node/>
-        </link>
-        <joint type="${gbeam_mate_joint_type}" name='n1l12'>
-          <pose>0 -2 0 0 0 0</pose>
-          <parent>node1</parent>
-          <child>link12</child>
-          <xacro:gbeam_mate/>
-        </joint>
-        <link name ='link12'>
-          <self_collide>1</self_collide>
-          <pose>0 2.5 .5 0 0 0</pose>
-          <xacro:gbeam_link/>
-        </link>
-        <joint type="${gbeam_mate_joint_type}" name='l12n2'>
-          <pose>0 2 0 0 0 0</pose>
-          <parent>node2</parent>
-          <child>link12</child>
-          <xacro:gbeam_mate/>
-        </joint>
-        <link name ='node2'>
-          <pose>0 5 0.5 0 0 0</pose>
-          <xacro:gbeam_node/>
-        </link>
-        <joint type="${gbeam_mate_joint_type}" name='n2l23'>
-          <pose>0 -2 0 0 0 0</pose>
-          <parent>node2</parent>
-          <child>link23</child>
-          <xacro:gbeam_mate/>
-        </joint>
-        <link name ='link23'>
-          <pose>0 5 3 ${pi/2.0} 0 0</pose>
-          <xacro:gbeam_link/>
-        </link>
-        <joint type="${gbeam_mate_joint_type}" name='l23n3'>
-          <pose>0 2 0 0 0 0</pose>
-          <parent>node3</parent>
-          <child>link23</child>
-          <xacro:gbeam_mate/>
-        </joint>
-        <link name ='node3'>
-          <pose>0 5 5.5 0 0 0</pose>
-          <xacro:gbeam_node/>
-        </link>
-        <joint type="${gbeam_mate_joint_type}" name='n3l34'>
-          <pose>0 2 0 0 0 0</pose>
-          <parent>node3</parent>
-          <child>link34</child>
-          <xacro:gbeam_mate/>
-        </joint>
-        <link name ='link34'>
-          <pose>0 2.5 5.5 0 0 0</pose>
-          <xacro:gbeam_link/>
-        </link>
-        <joint type="${gbeam_mate_joint_type}" name='l34n4'>
-          <pose>0 -2 0 0 0 0</pose>
-          <parent>node4</parent>
-          <child>link34</child>
-          <xacro:gbeam_mate/>
-        </joint>
-        <link name ='node4'>
-          <pose>0 0 5.5 0 0 0</pose>
-          <xacro:gbeam_node/>
-        </link>
-        <joint type="${gbeam_mate_joint_type}" name='n4l41'>
-          <pose>0 2 0 0 0 0</pose>
-          <parent>node4</parent>
-          <child>link41</child>
-          <xacro:gbeam_mate/>
-        </joint>
-        <link name ='link41'>
-          <pose>0 0 3 ${pi/2.0} 0 0</pose>
-          <xacro:gbeam_link/>
-        </link>
-        <joint type="${gbeam_mate_joint_type}" name='l41n1'>
-          <pose>0 -2 0 0 0 0</pose>
-          <parent>node1</parent>
-          <child>link41</child>
-          <xacro:gbeam_mate/>
-        </joint>
-      </model>
-    </xacro:if>
+   </xacro:if>
     <xacro:include filename="$(find gbeam_sim)/gbeam_soup.sdf.xacro"/>
   </world>

File: gbeam_sim/gbeam_soup.sdf.xacro (robot description, xacro)
@@ -60,4 +60,6 @@
   <model name="gbeam_soup">
     <plugin name="assembly_soup" filename="libassembly_soup_plugin.so">
+      <trans_mate_err>10.0</trans_mate_err>
+      <rot_mate_err>10.0</rot_mate_err>
       <!-- Mate Models -->
       <mate_model type="gbeam">

Commit message: Correct parsing of joint properties and correct joint creation
Also restoring old rviz integration

File: gbeam_sim/gbeam.world.xacro (robot description, xacro)
@@ -10,26 +10,26 @@
       <uri>model://ground_plane</uri>
     </include>
-    <xacro:if value="1">
-      <model name ='hog'>
-        <plugin name='hand_of_god' filename="libgazebo_ros_hand_of_god.so">
-          <frameId>hydra_right_grab</frameId>
-          <linkName>hog</linkName>
-        </plugin>
-        <link name ='hog'>
-          <self_collide>0</self_collide>
-          <pose>0 0 1 0 0 0</pose>
-          <collision name ='collision'>
-            <geometry>
-              <sphere><radius>0.025</radius></sphere>
-            </geometry>
-          </collision>
-          <visual name ='visual'>
-            <geometry>
-              <sphere><radius>0.025</radius></sphere>
-            </geometry>
-          </visual>
-        </link>
-      </model>
-   </xacro:if>
+    <!-- Hand of God -->
+    <model name ='hog'>
+      <plugin name='hand_of_god' filename="libgazebo_ros_hand_of_god.so">
+        <frameId>hog</frameId>
+        <linkName>hog</linkName>
+      </plugin>
+      <link name ='hog'>
+        <self_collide>0</self_collide>
+        <pose>0 0 1 0 0 0</pose>
+        <collision name ='collision'>
+          <geometry>
+            <sphere><radius>0.025</radius></sphere>
+          </geometry>
+        </collision>
+        <visual name ='visual'>
+          <geometry>
+            <sphere><radius>0.025</radius></sphere>
+          </geometry>
+        </visual>
+      </link>
+    </model>
+    <!-- GBeam Soup -->
     <xacro:include filename="$(find gbeam_sim)/gbeam_soup.sdf.xacro"/>
   </world>

File: gbeam_sim/gbeam_soup.sdf.xacro (robot description, xacro)
@@ -71,10 +71,10 @@
           <rot>1 1 4</rot>
         </symmetry>
-        <joint type="revolute" name="gbeam">
+        <joint type="prismatic" name="gbeam">
           <pose>0 0.025 0 0 ${pi/2} 0</pose>
           <parent>gbeam_link</parent>
           <child>gbeam_node</child>
           <axis>
-            <xyz>1 0 0</xyz>
+            <xyz>0 1 0</xyz>
             <limit><lower>-0.01</lower><upper>0.01</upper></limit>
           </axis>

Commit message: demo with multiple links and nodes

File: gbeam_sim/gbeam.world.xacro (robot description, xacro)
@@ -15,5 +15,5 @@
         <frameId>hog</frameId>
         <linkName>hog</linkName>
-        <kl>10000</kl>
+        <kl>400</kl>
         <ka>200</ka>
       </plugin>

File: gbeam_sim/gbeam_soup.sdf.xacro (robot description, xacro)
@@ -16,5 +16,5 @@
       <collision name='collision'>
         <geometry>
-          <mesh><uri>file://$(find gbeam_model)/meshes/gbeam_link_50k.dae</uri></mesh>
+          <mesh><uri>file://$(find gbeam_model)/meshes/gbeam_link_5k.stl</uri></mesh>
         </geometry>
         <surface>
@@ -29,5 +29,5 @@
       <visual name='visual'>
         <geometry>
-          <mesh><uri>file://$(find gbeam_model)/meshes/gbeam_link_50k.dae</uri></mesh>
+          <mesh><uri>file://$(find gbeam_model)/meshes/gbeam_link_5k.stl</uri></mesh>
         </geometry>
       </visual>
@@ -48,5 +48,5 @@
       <collision name='collision'>
         <geometry>
-          <mesh><uri>file://$(find gbeam_model)/meshes/gbeam_node_25k.dae</uri></mesh>
+          <mesh><uri>file://$(find gbeam_model)/meshes/gbeam_node_5k.stl</uri></mesh>
         </geometry>
         <surface>
@@ -61,5 +61,5 @@
       <visual name='visual'>
         <geometry>
-          <mesh><uri>file://$(find gbeam_model)/meshes/gbeam_node_25k.dae</uri></mesh>
+          <mesh><uri>file://$(find gbeam_model)/meshes/gbeam_node_5k.stl</uri></mesh>
         </geometry>
       </visual>
@@ -137,11 +137,11 @@
       </atom_model>
     </plugin>
-    <xacro:gbeam_node suffix="_1" pose="0 0.3 0.2 0 0 0"/>
-    <!--<xacro:gbeam_node suffix="_2" pose="0 0 0.1 0 0 0"/>-->
-    <!--<xacro:gbeam_node suffix="_3" pose="0 0 0.2 0 0 0"/>-->
+    <xacro:gbeam_node suffix="_1" pose="0 0.3 0.1 0 0 0"/>
+    <xacro:gbeam_node suffix="_2" pose="0 0.3 0.2 0 0 0"/>
+    <xacro:gbeam_node suffix="_3" pose="0 0.3 0.3 0 0 0"/>
     <!--<xacro:gbeam_node suffix="_4" pose="0 0 0.3 0 0 0"/>-->
     <!--<xacro:gbeam_node suffix="_5" pose="0 0 0.4 0 0 0"/>-->
     <xacro:gbeam_link suffix="_1" pose="0 0 0.2 0 0 0"/>
-    <!--<xacro:gbeam_link suffix="_2" pose="0 0.1 0.1 0 0 0"/>-->
+    <xacro:gbeam_link suffix="_2" pose="0.1 0.2 0.2 0 0 0"/>
     <!--<xacro:gbeam_link suffix="_3" pose="0 0.1 0.2 0 0 0"/>-->
     <!--<xacro:gbeam_link suffix="_4" pose="0 0.1 0.3 0 0 0"/>-->
