Commit message: now with mating hog

File: gbeam_sim/gbeam.world.xacro (robot description, xacro)
@@ -10,37 +10,42 @@
       <uri>model://ground_plane</uri>
     </include>
-    <!-- Hand of God -->
-    <model name ='hog'>
-      <plugin name='hand_of_god' filename="libgazebo_ros_hand_of_god.so">
-        <frameId>hog</frameId>
-        <linkName>hog</linkName>
-        <kl>400</kl>
-        <ka>200</ka>
-      </plugin>
-      <link name ='hog'>
-        <self_collide>0</self_collide>
-        <pose>0 0 1 0 0 0</pose>
-        <collision name ='collision'>
-          <geometry>
-            <sphere><radius>0.025</radius></sphere>
-          </geometry>
-        </collision>
-        <visual name ='visual'>
-          <geometry>
-            <sphere><radius>0.025</radius></sphere>
-          </geometry>
-        </visual>
-        <inertial>
-          <mass>0.3</mass>
-          <inertia>
-            <ixx>0.001</ixx><ixy>0</ixy>    <ixz>0</ixz>
-            <iyy>0.001</iyy><iyz>0</iyz>
-            <izz>0.001</izz>
-          </inertia>
-        </inertial>
-      </link>
-    </model>
+    <physics type="ode">
+      <gravity>0 0 -9.8</gravity>
+    </physics>
     <!-- GBeam Soup -->
     <xacro:include filename="$(find gbeam_sim)/gbeam_soup.sdf.xacro"/>
+    <!-- Hand of God -->
+    <xacro:if value="0">
+      <model name ='hog'>
+        <plugin name='hand_of_god' filename="libgazebo_ros_hand_of_god.so">
+          <frameId>hog</frameId>
+          <linkName>hog</linkName>
+          <kl>400</kl>
+          <ka>200</ka>
+        </plugin>
+        <link name ='hog'>
+          <self_collide>0</self_collide>
+          <pose>0 0 1 0 0 0</pose>
+          <collision name ='collision'>
+            <geometry>
+              <sphere><radius>0.025</radius></sphere>
+            </geometry>
+          </collision>
+          <visual name ='visual'>
+            <geometry>
+              <sphere><radius>0.025</radius></sphere>
+            </geometry>
+          </visual>
+          <inertial>
+            <mass>0.3</mass>
+            <inertia>
+              <ixx>0.001</ixx><ixy>0</ixy>    <ixz>0</ixz>
+              <iyy>0.001</iyy><iyz>0</iyz>
+              <izz>0.001</izz>
+            </inertia>
+          </inertial>
+        </link>
+      </model>
+    </xacro:if>
   </world>
 </sdf>

File: gbeam_sim/gbeam_soup.sdf.xacro (robot description, xacro)
@@ -4,6 +4,7 @@
   <xacro:macro name="gbeam_link" params="suffix pose">
     <link name="gbeam_link${suffix}">
+      <gravity>1</gravity>
+      <self_collide>1</self_collide>
       <pose>${pose}</pose>
-      <self_collide>1</self_collide>
       <inertial>
         <mass>0.3</mass>
@@ -36,6 +37,7 @@
   <xacro:macro name="gbeam_node" params="suffix pose">
     <link name="gbeam_node${suffix}">
+      <gravity>1</gravity>
+      <self_collide>1</self_collide>
       <pose>${pose}</pose>
-      <self_collide>1</self_collide>
       <inertial>
         <mass>0.2</mass>
@@ -67,4 +69,10 @@
   </xacro:macro>
   <model name="gbeam_soup">
+    <plugin name='hand_of_god' filename="libgazebo_ros_hand_of_god.so">
+      <frameId>hog</frameId>
+      <linkName>hog</linkName>
+      <kl>400</kl>
+      <ka>200</ka>
+    </plugin>
     <plugin name="assembly_soup" filename="libassembly_soup_plugin.so">
       <!-- Frame that poses are broadcasted in -->
@@ -92,10 +100,10 @@
           <axis>
             <xyz>0 1 0</xyz>
-            <limit><lower>-0.01</lower><upper>0.01</upper></limit>
+            <limit><lower>-0.001</lower><upper>0.001</upper></limit>
           </axis>
           <physics>
             <ode>
               <cfm_damping>true</cfm_damping>
-              <cfm>0.1</cfm>
+              <cfm>0.01</cfm>
               <erp>0.05</erp>
               <limit>
@@ -107,4 +115,43 @@
         </joint>
       </mate_model>
+      <!-- Experimental: add a mate point to the hog -->
+      <atom_model type="hog">
+        <mate_point type="gbeam" gender="female">
+          <pose>0 0.025 0 ${pi/2} 0 0</pose>
+        </mate_point>
+        <mate_point type="gbeam" gender="female">
+          <pose>0 -0.025 0 ${pi/2} 0 ${pi}</pose>
+        </mate_point>
+        <mate_point type="gbeam" gender="female">
+          <pose>0 0 0.025 ${pi} 0 0</pose>
+        </mate_point>
+        <mate_point type="gbeam" gender="female">
+          <pose>0 0 -0.025 0 0 0</pose>
+        </mate_point>
+        <mate_point type="gbeam" gender="female">
+          <pose>0.025 0 0 0 -${pi/2.0} 0</pose>
+        </mate_point>
+        <mate_point type="gbeam" gender="female">
+          <pose>-0.025 0 0 0 ${pi/2.0} 0</pose>
+        </mate_point>
+        <mate_point type="gbeam" gender="male">
+          <pose>0 -0.025 0 ${pi/2} 0 0</pose>
+        </mate_point>
+        <mate_point type="gbeam" gender="male">
+          <pose>0 0.025 0 ${pi/2} 0 ${pi}</pose>
+        </mate_point>
+        <mate_point type="gbeam" gender="male">
+          <pose>0 0 -0.025 ${pi} 0 0</pose>
+        </mate_point>
+        <mate_point type="gbeam" gender="male">
+          <pose>0 0 0.025 0 0 0</pose>
+        </mate_point>
+        <mate_point type="gbeam" gender="male">
+          <pose>-0.025 0 0 0 -${pi/2.0} 0</pose>
+        </mate_point>
+        <mate_point type="gbeam" gender="male">
+          <pose>0.025 0 0 0 ${pi/2.0} 0</pose>
+        </mate_point>
+      </atom_model>
       <!-- Atom Models -->
       <atom_model type="gbeam_link">
@@ -147,4 +194,26 @@
     <!--<xacro:gbeam_link suffix="_4" pose="0 0.1 0.3 0 0 0"/>-->
     <!--<xacro:gbeam_link suffix="_5" pose="0 0.1 0.4 0 0 0"/>-->
+    <link name ='hog'>
+      <self_collide>1</self_collide>
+      <pose>0 0 0.4 0 0 0</pose>
+      <collision name ='collision'>
+        <geometry>
+          <sphere><radius>0.025</radius></sphere>
+        </geometry>
+      </collision>
+      <visual name ='visual'>
+        <geometry>
+          <sphere><radius>0.025</radius></sphere>
+        </geometry>
+      </visual>
+      <inertial>
+        <mass>0.3</mass>
+        <inertia>
+          <ixx>0.001</ixx><ixy>0</ixy>    <ixz>0</ixz>
+          <iyy>0.001</iyy><iyz>0</iyz>
+          <izz>0.001</izz>
+        </inertia>
+      </inertial>
+    </link>
   </model>
 </sdf>
