Commit message: fixes for gazebo magnetic beams plugins: parsing joints now works correctly

File: gbeam_sim/gbeam_soup.sdf.xacro (robot description, xacro)
@@ -12,24 +12,28 @@
           <rot>1 1 4</rot>
         </symmetry>
-        <joint type="revolute1" name="gbeam">
-          <pose>0 0.5 0 0 ${pi/2} 0</pose>
-          <parent>gbeam_link</parent>
-          <child>gbeam_node</child>
-          <axis>
-            <xyz>1 0 0</xyz>
-            <limit><lower>0</lower><upper>0</upper></limit>
-          </axis>
-          <physics>
-            <ode>
-              <cfm_damping>1</cfm_damping>
-              <cfm>0.1</cfm>
-              <erp>0.1</erp>
-              <limit>
-                <cfm>0.1</cfm>
-                <erp>0.1</erp>
-              </limit>
-            </ode>
-          </physics>
-        </joint>
+          <sdf version="1.4">
+            <model name="template">
+              <joint type="revolute" name="gbeam">
+                <pose>0 0.5 0 0 ${pi/2} 0</pose>
+                <parent>gbeam_link</parent>
+                <child>gbeam_node</child>
+                <axis>
+                  <xyz>1 0 0</xyz>
+                  <limit><lower>0</lower><upper>0</upper></limit>
+                </axis>
+                <physics>
+                  <ode>
+                    <cfm_damping>1</cfm_damping>
+                    <cfm>0.1</cfm>
+                    <erp>0.1</erp>
+                    <limit>
+                      <cfm>0.1</cfm>
+                      <erp>0.1</erp>
+                    </limit>
+                  </ode>
+                </physics>
+              </joint>
+            </model>
+          </sdf>
       </mate_model>
       <!-- Atom Models -->

Commit message: gazebo does not want people to create models dynamically...

File: gbeam_sim/gbeam_soup.sdf.xacro (robot description, xacro)
@@ -12,28 +12,24 @@
           <rot>1 1 4</rot>
         </symmetry>
-          <sdf version="1.4">
-            <model name="template">
-              <joint type="revolute" name="gbeam">
-                <pose>0 0.5 0 0 ${pi/2} 0</pose>
-                <parent>gbeam_link</parent>
-                <child>gbeam_node</child>
-                <axis>
-                  <xyz>1 0 0</xyz>
-                  <limit><lower>0</lower><upper>0</upper></limit>
-                </axis>
-                <physics>
-                  <ode>
-                    <cfm_damping>1</cfm_damping>
-                    <cfm>0.1</cfm>
-                    <erp>0.1</erp>
-                    <limit>
-                      <cfm>0.1</cfm>
-                      <erp>0.1</erp>
-                    </limit>
-                  </ode>
-                </physics>
-              </joint>
-            </model>
-          </sdf>
+        <joint type="revolute" name="gbeam">
+          <pose>0 0.5 0 0 ${pi/2} 0</pose>
+          <parent>gbeam_link</parent>
+          <child>gbeam_node</child>
+          <axis>
+            <xyz>1 0 0</xyz>
+            <limit><lower>0</lower><upper>0</upper></limit>
+          </axis>
+          <physics>
+            <ode>
+              <cfm_damping>1</cfm_damping>
+              <cfm>0.1</cfm>
+              <erp>0.1</erp>
+              <limit>
+                <cfm>0.1</cfm>
+                <erp>0.1</erp>
+              </limit>
+            </ode>
+          </physics>
+        </joint>
       </mate_model>
       <!-- Atom Models -->

Commit message: updating assembly sim to statically create links, dynamically create joints

File: gbeam_sim/gbeam_soup.sdf.xacro (robot description, xacro)
@@ -2,4 +2,60 @@
 <sdf version="1.4" xmlns:xacro="http://www.ros.org/wiki/xacro" >
   <xacro:property name="pi" value="3.14159265"/>
+  <xacro:macro name="gbeam_link" params="suffix pose">
+    <link name="gbeam_link${suffix}">
+      <pose>${pose}</pose>
+      <self_collide>1</self_collide>
+      <inertial>
+        <mass>0.3</mass>
+        <inertia>
+          <ixx>0.001</ixx><ixy>0</ixy>    <ixz>0</ixz>
+          <iyy>0.002</iyy><iyz>0</iyz>
+          <izz>0.001</izz>
+        </inertia>
+      </inertial>
+      <collision name='collision'>
+        <geometry>
+          <box>
+            <size>0.05 0.3 0.05</size>
+          </box>
+        </geometry>
+      </collision>
+      <visual name='visual'>
+        <geometry>
+          <box>
+            <size>0.05 0.3 0.05</size>
+          </box>
+        </geometry>
+      </visual>
+    </link>
+  </xacro:macro>
+  <xacro:macro name="gbeam_node" params="suffix pose">
+    <link name="gbeam_node${suffix}">
+      <pose>${pose}</pose>
+      <self_collide>1</self_collide>
+      <inertial>
+        <mass>0.2</mass>
+        <inertia>
+          <ixx>0.001</ixx><ixy>0</ixy>    <ixz>0</ixz>
+          <iyy>0.001</iyy><iyz>0</iyz>
+          <izz>0.001</izz>
+        </inertia>
+      </inertial>
+      <collision name='collision'>
+        <geometry>
+          <box>
+            <size>0.05 0.05 0.05</size>
+          </box>
+        </geometry>
+      </collision>
+      <visual name='visual'>
+        <geometry>
+          <box>
+            <size>0.05 0.05 0.05</size>
+          </box>
+        </geometry>
+      </visual>
+    </link>
+  </xacro:macro>
   <model name="gbeam_soup">
     <plugin name="assembly_soup" filename="libassembly_soup_plugin.so">
@@ -35,110 +91,42 @@
       <!-- Atom Models -->
       <atom_model type="gbeam_link">
-        <link name="gbeam_link">
-          <pose>0 0 0 0 0 0</pose>
-          <self_collide>0</self_collide>
-          <inertial>
-            <mass>0.3</mass>
-            <inertia>
-              <ixx>0.001</ixx><ixy>0</ixy>    <ixz>0</ixz>
-                              <iyy>0.002</iyy><iyz>0</iyz>
-                                              <izz>0.001</izz>
-            </inertia>
-          </inertial>
-          <collision name='collision'>
-            <geometry>
-              <box>
-                <size>0.05 0.3 0.05</size>
-              </box>
-            </geometry>
-          </collision>
-          <visual name='visual'>
-            <geometry>
-              <box>
-                <size>0.05 0.3 0.05</size>
-              </box>
-            </geometry>
-          </visual>
-        </link>
         <mate_point type="gbeam" gender="male">
           <pose>0 0.100 0 ${pi/2.0} 0 0</pose>
         </mate_point>
-        <mate_point type="gbeam" gender="male">
-          <pose>0 -0.100 0 -${pi/2.0} 0 0</pose>
-        </mate_point>
+        <!--<mate_point type="gbeam" gender="male">-->
+          <!--<pose>0 -0.100 0 -${pi/2.0} 0 0</pose>-->
+        <!--</mate_point>-->
       </atom_model>
       <atom_model type="gbeam_node">
-        <link name="gbeam_node">
-          <pose>0 0 0 0 0 0</pose>
-          <self_collide>0</self_collide>
-          <inertial>
-            <mass>0.2</mass>
-            <inertia>
-              <ixx>0.001</ixx><ixy>0</ixy>    <ixz>0</ixz>
-                              <iyy>0.001</iyy><iyz>0</iyz>
-                                              <izz>0.001</izz>
-            </inertia>
-          </inertial>
-          <collision name='collision'>
-            <geometry>
-              <box>
-                <size>0.05 0.05 0.05</size>
-              </box>
-            </geometry>
-          </collision>
-          <visual name='visual'>
-            <geometry>
-              <box>
-                <size>0.05 0.05 0.05</size>
-              </box>
-            </geometry>
-          </visual>
-        </link>
         <mate_point type="gbeam" gender="female">
           <pose>0 0 0.5 0 0 0</pose>
         </mate_point>
-        <mate_point type="gbeam" gender="female">
-          <pose>0 0 -0.05 0 0 ${pi}</pose>
-        </mate_point>
-        <mate_point type="gbeam" gender="female">
-          <pose>0 0.05 0 -${pi/2.0} 0 0</pose>
-        </mate_point>
-        <mate_point type="gbeam" gender="female">
-          <pose>0 -0.05 0 ${pi/2.0} 0 0</pose>
-        </mate_point>
-        <mate_point type="gbeam" gender="female">
-          <pose>0.05 0 0 0 ${pi/2.0} 0</pose>
-        </mate_point>
-        <mate_point type="gbeam" gender="female">
-          <pose>-0.05 0 0 0 -${pi/2.0} 0</pose>
-        </mate_point>
+        <!--<mate_point type="gbeam" gender="female">-->
+          <!--<pose>0 0 -0.05 0 0 ${pi}</pose>-->
+        <!--</mate_point>-->
+        <!--<mate_point type="gbeam" gender="female">-->
+          <!--<pose>0 0.05 0 -${pi/2.0} 0 0</pose>-->
+        <!--</mate_point>-->
+        <!--<mate_point type="gbeam" gender="female">-->
+          <!--<pose>0 -0.05 0 ${pi/2.0} 0 0</pose>-->
+        <!--</mate_point>-->
+        <!--<mate_point type="gbeam" gender="female">-->
+          <!--<pose>0.05 0 0 0 ${pi/2.0} 0</pose>-->
+        <!--</mate_point>-->
+        <!--<mate_point type="gbeam" gender="female">-->
+          <!--<pose>-0.05 0 0 0 -${pi/2.0} 0</pose>-->
+        <!--</mate_point>-->
       </atom_model>
-      <assembly>
-        <atom type="gbeam_node">
-          <pose>0 0 0 0 0 0</pose>
-        </atom>
-        <atom type="gbeam_node">
-          <pose>0 0 0.3 0 0 0</pose>
-        </atom>
-        <atom type="gbeam_node">
-          <pose>0 0 0.6 0 0 0</pose>
-        </atom>
-        <atom type="gbeam_node">
-          <pose>0 0 0.9 0 0 0</pose>
-        </atom>
-        <atom type="gbeam_link">
-          <pose>0 0 0 0 0 0</pose>
-        </atom>
-        <atom type="gbeam_link">
-          <pose>0 0 0.1 0 0 0</pose>
-        </atom>
-        <atom type="gbeam_link">
-          <pose>0 0 0.2 0 0 0</pose>
-        </atom>
-        <atom type="gbeam_link">
-          <pose>0 0 0.3 0 0 0</pose>
-        </atom>
-      </assembly>
     </plugin>
+    <xacro:gbeam_node suffix="_1" pose="0 0 0 0 0 0"/>
+    <!--<xacro:gbeam_node suffix="_2" pose="0 0 0.1 0 0 0"/>-->
+    <!--<xacro:gbeam_node suffix="_3" pose="0 0 0.2 0 0 0"/>-->
+    <!--<xacro:gbeam_node suffix="_4" pose="0 0 0.3 0 0 0"/>-->
+    <!--<xacro:gbeam_node suffix="_5" pose="0 0 0.4 0 0 0"/>-->
+    <xacro:gbeam_link suffix="_1" pose="0 0.3 0 0 0 0"/>
+    <!--<xacro:gbeam_link suffix="_2" pose="0 0.1 0.1 0 0 0"/>-->
+    <!--<xacro:gbeam_link suffix="_3" pose="0 0.1 0.2 0 0 0"/>-->
+    <!--<xacro:gbeam_link suffix="_4" pose="0 0.1 0.3 0 0 0"/>-->
+    <!--<xacro:gbeam_link suffix="_5" pose="0 0.1 0.4 0 0 0"/>-->
   </model>
 </sdf>

Commit message: experimented with attaching joints; everything works a little bit better now

File: gbeam_sim/gbeam_soup.sdf.xacro (robot description, xacro)
@@ -60,5 +60,5 @@
   <model name="gbeam_soup">
     <plugin name="assembly_soup" filename="libassembly_soup_plugin.so">
-      <trans_mate_err>0.2</trans_mate_err>
+      <trans_mate_err>0.01</trans_mate_err>
       <rot_mate_err>0.1</rot_mate_err>
       <tf_world_frame>world</tf_world_frame>
@@ -77,14 +77,14 @@
           <axis>
             <xyz>1 0 0</xyz>
-            <limit><lower>0</lower><upper>0</upper></limit>
+            <limit><lower>-0.01</lower><upper>0.01</upper></limit>
           </axis>
           <physics>
             <ode>
               <cfm_damping>true</cfm_damping>
-              <cfm>0.2</cfm>
+              <cfm>0.1</cfm>
               <erp>0.05</erp>
               <limit>
                 <cfm>0.1</cfm>
-                <erp>0.2</erp>
+                <erp>0.5</erp>
               </limit>
             </ode>

Commit message: moved definitions to a new file to make experiments easier

File: gbeam_sim/gbeam_soup.sdf.xacro (robot description, xacro)
@@ -1,83 +1,5 @@
 <?xml version='1.0'?>
 <sdf version="1.4" xmlns:xacro="http://www.ros.org/wiki/xacro" >
-  <xacro:property name="pi" value="3.14159265"/>
-  <xacro:macro name="gbeam_link" params="suffix pose">
-    <link name="gbeam_link${suffix}">
-      <gravity>1</gravity>
-      <self_collide>1</self_collide>
-      <pose>${pose}</pose>
-      <inertial>
-        <mass>0.3</mass>
-        <inertia>
-          <ixx>0.001</ixx><ixy>0</ixy>    <ixz>0</ixz>
-          <iyy>0.002</iyy><iyz>0</iyz>
-          <izz>0.001</izz>
-        </inertia>
-      </inertial>
-      <collision name='collision'>
-        <geometry>
-          <mesh><uri>file://$(find gbeam_model)/meshes/gbeam_link_5k.stl</uri></mesh>
-        </geometry>
-        <surface>
-          <friction>
-            <ode>
-              <mu>1.0</mu>
-              <mu2>0.7</mu2>
-            </ode>
-          </friction>
-          <contact>
-            <ode>
-              <soft_cfm>0.01</soft_cfm>
-              <soft_erp>0.05</soft_erp>
-            </ode>
-          </contact>
-        </surface>
-      </collision>
-      <visual name='visual'>
-        <geometry>
-          <mesh><uri>file://$(find gbeam_model)/meshes/gbeam_link_5k.stl</uri></mesh>
-        </geometry>
-      </visual>
-    </link>
-  </xacro:macro>
-  <xacro:macro name="gbeam_node" params="suffix pose">
-    <link name="gbeam_node${suffix}">
-      <gravity>1</gravity>
-      <self_collide>1</self_collide>
-      <pose>${pose}</pose>
-      <inertial>
-        <mass>0.2</mass>
-        <inertia>
-          <ixx>0.001</ixx><ixy>0</ixy>    <ixz>0</ixz>
-          <iyy>0.001</iyy><iyz>0</iyz>
-          <izz>0.001</izz>
-        </inertia>
-      </inertial>
-      <collision name='collision'>
-        <geometry>
-          <mesh><uri>file://$(find gbeam_model)/meshes/gbeam_node_5k.stl</uri></mesh>
-        </geometry>
-        <surface>
-          <friction>
-            <ode>
-              <mu>0.5</mu>
-              <mu2>0.5</mu2>
-            </ode>
-          </friction>
-          <contact>
-            <ode>
-              <soft_cfm>0.01</soft_cfm>
-              <soft_erp>0.05</soft_erp>
-            </ode>
-          </contact>
-        </surface>
-      </collision>
-      <visual name='visual'>
-        <geometry>
-          <mesh><uri>file://$(find gbeam_model)/meshes/gbeam_node_5k.stl</uri></mesh>
-        </geometry>
-      </visual>
-    </link>
-  </xacro:macro>
+  <xacro:include filename="$(find gbeam_sim)/gbeam_def.sdf.xacro"/>
   <model name="gbeam_soup">
     <plugin name='hand_of_god' filename="libgazebo_ros_hand_of_god.so">
@@ -91,40 +13,9 @@
       <tf_world_frame>world</tf_world_frame>
       <!-- Mate Models -->
-      <mate_model type="gbeam">
-        <!-- planar shear-supporting magnetic mate
-             mating surface is along positive z-axis
-             -->
-        <symmetry>
-          <rot>1 1 4</rot>
-        </symmetry>
-        <attach_threshold>
-          <linear>0.004</linear>
-          <angular>0.1</angular>
-        </attach_threshold>
-        <detach_threshold>
-          <linear>0.015</linear>
-          <angular>0.2</angular>
-        </detach_threshold>
-        <joint type="prismatic" name="gbeam">
-          <pose>0 0.025 0 0 ${pi/2} 0</pose>
-          <parent>gbeam_link</parent>
-          <child>gbeam_node</child>
-          <axis>
-            <xyz>0 1 0</xyz>
-            <limit><lower>-0.001</lower><upper>0.001</upper></limit>
-          </axis>
-          <physics>
-            <ode>
-              <cfm_damping>true</cfm_damping>
-              <cfm>0.01</cfm>
-              <erp>0.05</erp>
-              <limit>
-                <cfm>0.1</cfm>
-                <erp>0.5</erp>
-              </limit>
-            </ode>
-          </physics>
-        </joint>
-      </mate_model>
+      <xacro:gbeam_mate
+        linear_attach="0.004"
+        angular_attach="0.1"
+        linear_detach="0.015"
+        angular_detach="0.2"/>
       <!-- Experimental: add a mate point to the hog -->
       <atom_model type="hog">
@@ -167,32 +58,6 @@
       </atom_model>
       <!-- Atom Models -->
-      <atom_model type="gbeam_link">
-        <mate_point type="gbeam" gender="male">
-          <pose>0 0.125 0 ${pi/2} ${pi/4} ${pi}</pose>
-        </mate_point>
-        <mate_point type="gbeam" gender="male">
-          <pose>0 -0.125 0 ${pi/2} ${pi/4} 0</pose>
-        </mate_point>
-      </atom_model>
-      <atom_model type="gbeam_node">
-        <mate_point type="gbeam" gender="female">
-          <pose>0 0.025 0 ${pi/2} 0 0</pose>
-        </mate_point>
-        <mate_point type="gbeam" gender="female">
-          <pose>0 -0.025 0 ${pi/2} 0 ${pi}</pose>
-        </mate_point>
-        <mate_point type="gbeam" gender="female">
-          <pose>0 0 0.025 ${pi} 0 0</pose>
-        </mate_point>
-        <mate_point type="gbeam" gender="female">
-          <pose>0 0 -0.025 0 0 0</pose>
-        </mate_point>
-        <mate_point type="gbeam" gender="female">
-          <pose>0.025 0 0 0 -${pi/2.0} 0</pose>
-        </mate_point>
-        <mate_point type="gbeam" gender="female">
-          <pose>-0.025 0 0 0 ${pi/2.0} 0</pose>
-        </mate_point>
-      </atom_model>
+      <xacro:gbeam_link_atom/>
+      <xacro:gbeam_node_atom/>
     </plugin>
     <xacro:gbeam_node suffix="_1" pose="0 0.3 0.1 0 0 0"/>
