Commit message: changed blocks to simplify collision meshes

File: gbeam_sim/gbeam_def.sdf.xacro (robot description, xacro)
@@ -15,23 +15,96 @@
         </inertia>
       </inertial>
-      <collision name='collision'>
-        <geometry>
-          <mesh><uri>file://$(find gbeam_model)/meshes/gbeam_link_5k.stl</uri></mesh>
-        </geometry>
-        <surface>
-          <friction>
-            <ode>
-              <mu>1.0</mu>
-              <mu2>0.7</mu2>
-            </ode>
-          </friction>
-          <contact>
-            <ode>
-              <soft_cfm>0.01</soft_cfm>
-              <soft_erp>0.05</soft_erp>
-            </ode>
-          </contact>
-        </surface>
-      </collision>
+      <xacro:unless value="true">
+        <collision name='collision'>
+          <!-- use full scanned collision mesh -->
+          <geometry>
+            <mesh><uri>file://$(find gbeam_model)/meshes/gbeam_link_5k.stl</uri></mesh>
+          </geometry>
+          <surface>
+            <friction>
+              <ode>
+                <mu>1.0</mu>
+                <mu2>0.7</mu2>
+              </ode>
+            </friction>
+            <contact>
+              <ode>
+                <soft_cfm>0.01</soft_cfm>
+                <soft_erp>0.05</soft_erp>
+              </ode>
+            </contact>
+          </surface>
+        </collision>
+      </xacro:unless>
+      <xacro:if value="true">
+        <collision name='gbeam_link_collision'>
+          <pose>0 0 0 0 -0 0</pose>
+          <geometry>
+            <box>
+              <size>0.035 0.24 0.035</size>
+            </box>
+          </geometry>
+          <surface>
+            <friction>
+              <ode>
+                <mu>1.0</mu>
+                <mu2>0.7</mu2>
+              </ode>
+            </friction>
+            <contact>
+              <ode>
+                <soft_cfm>0.01</soft_cfm>
+                <soft_erp>0.05</soft_erp>
+              </ode>
+            </contact>
+          </surface>
+        </collision>
+        <collision name='gbeam_link_collision_gbeam_link_1'>
+          <pose>0 0.115 0 1.5707 -0 0</pose>
+          <geometry>
+            <cylinder>
+              <length>0.0127</length>
+              <radius>0.028</radius>
+            </cylinder>
+          </geometry>
+          <surface>
+            <friction>
+              <ode>
+                <mu>1.0</mu>
+                <mu2>0.7</mu2>
+              </ode>
+            </friction>
+            <contact>
+              <ode>
+                <soft_cfm>0.01</soft_cfm>
+                <soft_erp>0.05</soft_erp>
+              </ode>
+            </contact>
+          </surface>
+        </collision>
+        <collision name='gbeam_link_collision_gbeam_link_2'>
+          <pose>0 -0.115 0 1.5707 -0 0</pose>
+          <geometry>
+            <cylinder>
+              <length>0.0127</length>
+              <radius>0.028</radius>
+            </cylinder>
+          </geometry>
+          <surface>
+            <friction>
+              <ode>
+                <mu>1.0</mu>
+                <mu2>0.7</mu2>
+              </ode>
+            </friction>
+            <contact>
+              <ode>
+                <soft_cfm>0.01</soft_cfm>
+                <soft_erp>0.05</soft_erp>
+              </ode>
+            </contact>
+          </surface>
+        </collision>
+      </xacro:if>
       <visual name='visual'>
         <geometry>

Commit message: cleaning up gbeam_sim

File: gbeam_sim/gbeam_def.sdf.xacro (robot description, xacro)
@@ -2,4 +2,5 @@
 <sdf version="1.4" xmlns:xacro="http://www.ros.org/wiki/xacro" >
   <xacro:property name="pi" value="3.14159265"/>
+  <!-- GBeam links -->
   <xacro:macro name="gbeam_link" params="suffix pose">
     <link name="gbeam_link${suffix}">
@@ -153,8 +154,39 @@
     </link>
   </xacro:macro>
+  <xacro:macro name="gbeam_hog" params="pose">
+    <plugin name='hand_of_god' filename="libgazebo_ros_hand_of_god.so">
+      <frameId>hog</frameId>
+      <linkName>hog</linkName>
+      <kl>400</kl>
+      <ka>200</ka>
+    </plugin>
+    <link name ='hog'>
+      <self_collide>1</self_collide>
+      <pose>${pose}</pose>
+      <collision name ='collision'>
+        <geometry>
+          <sphere><radius>0.025</radius></sphere>
+        </geometry>
+      </collision>
+      <visual name ='visual'>
+        <geometry>
+          <sphere><radius>0.025</radius></sphere>
+        </geometry>
+      </visual>
+      <inertial>
+        <mass>0.3</mass>
+        <inertia>
+          <ixx>0.001</ixx><ixy>0</ixy>    <ixz>0</ixz>
+          <iyy>0.001</iyy><iyz>0</iyz>
+          <izz>0.001</izz>
+        </inertia>
+      </inertial>
+    </link>
+  </xacro:macro>
+  <!-- GBeam mates -->
   <xacro:macro name="gbeam_mate" params="linear_attach angular_attach linear_detach angular_detach">
     <mate_model type="gbeam">
       <!-- planar shear-supporting magnetic mate
-             mating surface is along positive z-axis
+           mating surface is along positive z-axis
              -->
         <symmetry>
@@ -189,37 +221,78 @@
           </physics>
         </joint>
-      </mate_model>
-    </xacro:macro>
-    <xacro:macro name="gbeam_link_atom" params="">
-      <atom_model type="gbeam_link">
-        <mate_point type="gbeam" gender="male">
-          <pose>0 0.125 0 ${pi/2} ${pi/4} ${pi}</pose>
-        </mate_point>
-        <mate_point type="gbeam" gender="male">
-          <pose>0 -0.125 0 ${pi/2} ${pi/4} 0</pose>
-        </mate_point>
-      </atom_model>
-    </xacro:macro>
-    <xacro:macro name="gbeam_node_atom" params="">
-      <atom_model type="gbeam_node">
-        <mate_point type="gbeam" gender="female">
-          <pose>0 0.025 0 ${pi/2} 0 0</pose>
-        </mate_point>
-        <mate_point type="gbeam" gender="female">
-          <pose>0 -0.025 0 ${pi/2} 0 ${pi}</pose>
-        </mate_point>
-        <mate_point type="gbeam" gender="female">
-          <pose>0 0 0.025 ${pi} 0 0</pose>
-        </mate_point>
-        <mate_point type="gbeam" gender="female">
-          <pose>0 0 -0.025 0 0 0</pose>
-        </mate_point>
-        <mate_point type="gbeam" gender="female">
-          <pose>0.025 0 0 0 -${pi/2.0} 0</pose>
-        </mate_point>
-        <mate_point type="gbeam" gender="female">
-          <pose>-0.025 0 0 0 ${pi/2.0} 0</pose>
-        </mate_point>
-      </atom_model>
-    </xacro:macro>
-  </sdf>
+    </mate_model>
+  </xacro:macro>
+  <!-- GBeam atoms -->
+  <xacro:macro name="gbeam_link_atom" params="">
+    <atom_model type="gbeam_link">
+      <mate_point type="gbeam" gender="male">
+        <pose>0 0.125 0 ${pi/2} ${pi/4} ${pi}</pose>
+      </mate_point>
+      <mate_point type="gbeam" gender="male">
+        <pose>0 -0.125 0 ${pi/2} ${pi/4} 0</pose>
+      </mate_point>
+    </atom_model>
+  </xacro:macro>
+  <xacro:macro name="gbeam_node_atom" params="">
+    <atom_model type="gbeam_node">
+      <mate_point type="gbeam" gender="female">
+        <pose>0 0.025 0 ${pi/2} 0 0</pose>
+      </mate_point>
+      <mate_point type="gbeam" gender="female">
+        <pose>0 -0.025 0 ${pi/2} 0 ${pi}</pose>
+      </mate_point>
+      <mate_point type="gbeam" gender="female">
+        <pose>0 0 0.025 ${pi} 0 0</pose>
+      </mate_point>
+      <mate_point type="gbeam" gender="female">
+        <pose>0 0 -0.025 0 0 0</pose>
+      </mate_point>
+      <mate_point type="gbeam" gender="female">
+        <pose>0.025 0 0 0 -${pi/2.0} 0</pose>
+      </mate_point>
+      <mate_point type="gbeam" gender="female">
+        <pose>-0.025 0 0 0 ${pi/2.0} 0</pose>
+      </mate_point>
+    </atom_model>
+  </xacro:macro>
+  <xacro:macro name="gbeam_hog_atom" params="">
+    <atom_model type="hog">
+      <mate_point type="gbeam" gender="female">
+        <pose>0 0.025 0 ${pi/2} 0 0</pose>
+      </mate_point>
+      <mate_point type="gbeam" gender="female">
+        <pose>0 -0.025 0 ${pi/2} 0 ${pi}</pose>
+      </mate_point>
+      <mate_point type="gbeam" gender="female">
+        <pose>0 0 0.025 ${pi} 0 0</pose>
+      </mate_point>
+      <mate_point type="gbeam" gender="female">
+        <pose>0 0 -0.025 0 0 0</pose>
+      </mate_point>
+      <mate_point type="gbeam" gender="female">
+        <pose>0.025 0 0 0 -${pi/2.0} 0</pose>
+      </mate_point>
+      <mate_point type="gbeam" gender="female">
+        <pose>-0.025 0 0 0 ${pi/2.0} 0</pose>
+      </mate_point>
+      <mate_point type="gbeam" gender="male">
+        <pose>0 -0.025 0 ${pi/2} 0 0</pose>
+      </mate_point>
+      <mate_point type="gbeam" gender="male">
+        <pose>0 0.025 0 ${pi/2} 0 ${pi}</pose>
+      </mate_point>
+      <mate_point type="gbeam" gender="male">
+        <pose>0 0 -0.025 ${pi} 0 0</pose>
+      </mate_point>
+      <mate_point type="gbeam" gender="male">
+        <pose>0 0 0.025 0 0 0</pose>
+      </mate_point>
+      <mate_point type="gbeam" gender="male">
+        <pose>-0.025 0 0 0 -${pi/2.0} 0</pose>
+      </mate_point>
+      <mate_point type="gbeam" gender="male">
+        <pose>0.025 0 0 0 ${pi/2.0} 0</pose>
+      </mate_point>
+    </atom_model>
+  </xacro:macro>
+</sdf>

File: gbeam_sim/gbeam_soup.sdf.xacro (robot description, xacro)
@@ -3,14 +3,8 @@
   <xacro:include filename="$(find gbeam_sim)/gbeam_def.sdf.xacro"/>
   <model name="gbeam_soup">
-    <plugin name='hand_of_god' filename="libgazebo_ros_hand_of_god.so">
-      <frameId>hog</frameId>
-      <linkName>hog</linkName>
-      <kl>400</kl>
-      <ka>200</ka>
-    </plugin>
     <plugin name="assembly_soup" filename="libassembly_soup_plugin.so">
       <!-- Frame that poses are broadcasted in -->
       <tf_world_frame>world</tf_world_frame>
-      <!-- do we want to publish a list of joined mates for analysis? -->
+      <!--Publish a list of joined mates for analysis -->
       <publish_active_mates>1</publish_active_mates>
       <!-- Mate Models -->
@@ -20,47 +14,12 @@
         linear_detach="0.015"
         angular_detach="0.2"/>
-      <!-- Experimental: add a mate point to the hog -->
-      <atom_model type="hog">
-        <mate_point type="gbeam" gender="female">
-          <pose>0 0.025 0 ${pi/2} 0 0</pose>
-        </mate_point>
-        <mate_point type="gbeam" gender="female">
-          <pose>0 -0.025 0 ${pi/2} 0 ${pi}</pose>
-        </mate_point>
-        <mate_point type="gbeam" gender="female">
-          <pose>0 0 0.025 ${pi} 0 0</pose>
-        </mate_point>
-        <mate_point type="gbeam" gender="female">
-          <pose>0 0 -0.025 0 0 0</pose>
-        </mate_point>
-        <mate_point type="gbeam" gender="female">
-          <pose>0.025 0 0 0 -${pi/2.0} 0</pose>
-        </mate_point>
-        <mate_point type="gbeam" gender="female">
-          <pose>-0.025 0 0 0 ${pi/2.0} 0</pose>
-        </mate_point>
-        <mate_point type="gbeam" gender="male">
-          <pose>0 -0.025 0 ${pi/2} 0 0</pose>
-        </mate_point>
-        <mate_point type="gbeam" gender="male">
-          <pose>0 0.025 0 ${pi/2} 0 ${pi}</pose>
-        </mate_point>
-        <mate_point type="gbeam" gender="male">
-          <pose>0 0 -0.025 ${pi} 0 0</pose>
-        </mate_point>
-        <mate_point type="gbeam" gender="male">
-          <pose>0 0 0.025 0 0 0</pose>
-        </mate_point>
-        <mate_point type="gbeam" gender="male">
-          <pose>-0.025 0 0 0 -${pi/2.0} 0</pose>
-        </mate_point>
-        <mate_point type="gbeam" gender="male">
-          <pose>0.025 0 0 0 ${pi/2.0} 0</pose>
-        </mate_point>
-      </atom_model>
       <!-- Atom Models -->
       <xacro:gbeam_link_atom/>
       <xacro:gbeam_node_atom/>
+      <xacro:gbeam_hog_atom/>
     </plugin>
+    <!-- By adding a HOG to the soup, you can interact with the objects via mate points -->
+    <xacro:gbeam_hog pose="0 0 0.4 0 0 0"/>
+    <!-- Create the initial scene made of links and nodes -->
     <xacro:gbeam_node suffix="_1" pose="0 0.3 0.1 0 0 0"/>
     <xacro:gbeam_node suffix="_2" pose="0 0.3 0.2 0 0 0"/>
@@ -73,26 +32,4 @@
     <!--<xacro:gbeam_link suffix="_4" pose="0 0.1 0.3 0 0 0"/>-->
     <!--<xacro:gbeam_link suffix="_5" pose="0 0.1 0.4 0 0 0"/>-->
-    <link name ='hog'>
-      <self_collide>1</self_collide>
-      <pose>0 0 0.4 0 0 0</pose>
-      <collision name ='collision'>
-        <geometry>
-          <sphere><radius>0.025</radius></sphere>
-        </geometry>
-      </collision>
-      <visual name ='visual'>
-        <geometry>
-          <sphere><radius>0.025</radius></sphere>
-        </geometry>
-      </visual>
-      <inertial>
-        <mass>0.3</mass>
-        <inertia>
-          <ixx>0.001</ixx><ixy>0</ixy>    <ixz>0</ixz>
-          <iyy>0.001</iyy><iyz>0</iyz>
-          <izz>0.001</izz>
-        </inertia>
-      </inertial>
-    </link>
   </model>
 </sdf>

Commit message: adding visual appearances

File: gbeam_sim/gbeam_def.sdf.xacro (robot description, xacro)
@@ -25,12 +25,17 @@
             <friction>
               <ode>
-                <mu>1.0</mu>
-                <mu2>0.7</mu2>
+                <mu>0.7</mu>
+                <!--<mu2>0.7</mu2>-->
               </ode>
             </friction>
+            <bounce>
+              <restitution_coefficient>0.0</restitution_coefficient>
+            </bounce>
             <contact>
               <ode>
                 <soft_cfm>0.01</soft_cfm>
                 <soft_erp>0.05</soft_erp>
+                <kp>50000</kp>
+                <kd>8</kd>
               </ode>
             </contact>
@@ -43,5 +48,5 @@
           <geometry>
             <box>
-              <size>0.035 0.24 0.035</size>
+              <size>0.035 ${0.24+0.004} 0.035</size>
             </box>
           </geometry>
@@ -49,12 +54,17 @@
             <friction>
               <ode>
-                <mu>1.0</mu>
-                <mu2>0.7</mu2>
+                <mu>0.7</mu>
+                <!--<mu2>0.7</mu2>-->
               </ode>
             </friction>
+            <bounce>
+              <restitution_coefficient>0.0</restitution_coefficient>
+            </bounce>
             <contact>
               <ode>
                 <soft_cfm>0.01</soft_cfm>
                 <soft_erp>0.05</soft_erp>
+                <kp>50000</kp>
+                <kd>8</kd>
               </ode>
             </contact>
@@ -62,8 +72,8 @@
         </collision>
         <collision name='gbeam_link_collision_gbeam_link_1'>
-          <pose>0 0.115 0 1.5707 -0 0</pose>
+          <pose>0 ${0.115-0.00635/2.0} 0 1.5707 -0 0</pose>
           <geometry>
             <cylinder>
-              <length>0.0127</length>
+              <length>0.00635</length>
               <radius>0.028</radius>
             </cylinder>
@@ -72,6 +82,8 @@
             <friction>
               <ode>
-                <mu>1.0</mu>
-                <mu2>0.7</mu2>
+                <mu>1.7</mu>
+                <!--<mu2>0.7</mu2>-->
+                <slip1>1.0</slip1>
+                <slip2>1.0</slip2>
               </ode>
             </friction>
@@ -85,8 +97,8 @@
         </collision>
         <collision name='gbeam_link_collision_gbeam_link_2'>
-          <pose>0 -0.115 0 1.5707 -0 0</pose>
+          <pose>0 ${-0.115+0.00635/2.0} 0 1.5707 -0 0</pose>
           <geometry>
             <cylinder>
-              <length>0.0127</length>
+              <length>0.00635</length>
               <radius>0.028</radius>
             </cylinder>
@@ -95,12 +107,19 @@
             <friction>
               <ode>
-                <mu>1.0</mu>
-                <mu2>0.7</mu2>
+                <mu>1.7</mu>
+                <slip1>1.0</slip1>
+                <slip2>1.0</slip2>
+                <!--<mu2>0.7</mu2>-->
               </ode>
             </friction>
+            <bounce>
+              <restitution_coefficient>0.0</restitution_coefficient>
+            </bounce>
             <contact>
               <ode>
                 <soft_cfm>0.01</soft_cfm>
-                <soft_erp>0.05</soft_erp>
+                <soft_erp>0.02</soft_erp>
+                <kp>50000</kp>
+                <kd>8</kd>
               </ode>
             </contact>
@@ -109,6 +128,12 @@
       </xacro:if>
       <visual name='visual'>
-        <geometry>
-          <mesh><uri>file://$(find gbeam_model)/meshes/gbeam_link_5k.stl</uri></mesh>
+        <material>
+          <ambient>0.6 0.6 0.6 1</ambient>
+          <diffuse>0.5 0.5 0.5 1</diffuse>
+          <specular>1.0 1.0 1.0 1</specular>
+          <emissive>0 0 0 0</emissive>
+        </material>
+        <geometry>
+          <mesh><uri>file://$(find gbeam_model)/meshes/gbeam_link_visual.dae</uri></mesh>
         </geometry>
       </visual>
@@ -130,5 +155,6 @@
       <collision name='collision'>
         <geometry>
-          <mesh><uri>file://$(find gbeam_model)/meshes/gbeam_node_5k.stl</uri></mesh>
+          <!--<mesh><uri>file://$(find gbeam_model)/meshes/gbeam_node_5k.stl</uri></mesh>-->
+          <box><size>0.056 0.056 0.056</size></box>
         </geometry>
         <surface>
@@ -136,11 +162,16 @@
             <ode>
               <mu>0.5</mu>
-              <mu2>0.5</mu2>
+              <!--<mu2>0.5</mu2>-->
             </ode>
           </friction>
+          <bounce>
+            <restitution_coefficient>0.0</restitution_coefficient>
+          </bounce>
           <contact>
             <ode>
               <soft_cfm>0.01</soft_cfm>
-              <soft_erp>0.05</soft_erp>
+              <soft_erp>0.02</soft_erp>
+              <kp>50000</kp>
+              <kd>8</kd>
             </ode>
           </contact>
@@ -148,6 +179,12 @@
       </collision>
       <visual name='visual'>
-        <geometry>
-          <mesh><uri>file://$(find gbeam_model)/meshes/gbeam_node_5k.stl</uri></mesh>
+        <material>
+          <ambient>0.3 0.3 0.3 1</ambient>
+          <diffuse>0.5 0.5 0.5 1</diffuse>
+          <specular>1.0 1.0 1.0 1</specular>
+          <emissive>0 0 0 0</emissive>
+        </material>
+        <geometry>
+          <mesh><uri>file://$(find gbeam_model)/meshes/gbeam_node_visual.dae</uri></mesh>
         </geometry>
       </visual>
@@ -207,5 +244,8 @@
           <axis>
             <xyz>0 1 0</xyz>
-            <limit><lower>-0.001</lower><upper>0.001</upper></limit>
+            <limit>
+              <lower>-0.001</lower>
+              <upper>0.001</upper>
+            </limit>
           </axis>
           <physics>
@@ -215,6 +255,6 @@
               <erp>0.05</erp>
               <limit>
-                <cfm>0.1</cfm>
-                <erp>0.5</erp>
+                <cfm>0.05</cfm>
+                <erp>0.05</erp>
               </limit>
             </ode>
@@ -227,8 +267,8 @@
     <atom_model type="gbeam_link">
       <mate_point type="gbeam" gender="male">
-        <pose>0 0.125 0 ${pi/2} ${pi/4} ${pi}</pose>
-      </mate_point>
-      <mate_point type="gbeam" gender="male">
-        <pose>0 -0.125 0 ${pi/2} ${pi/4} 0</pose>
+        <pose>0 0.126 0 ${pi/2} ${pi/4} ${pi}</pose>
+      </mate_point>
+      <mate_point type="gbeam" gender="male">
+        <pose>0 -0.126 0 ${pi/2} ${pi/4} 0</pose>
       </mate_point>
     </atom_model>

File: gbeam_sim/gbeam_soup.sdf.xacro (robot description, xacro)
@@ -12,6 +12,6 @@
         linear_attach="0.004"
         angular_attach="0.1"
-        linear_detach="0.015"
-        angular_detach="0.2"/>
+        linear_detach="0.008"
+        angular_detach="0.15"/>
       <!-- Atom Models -->
       <xacro:gbeam_link_atom/>

Commit message: more accurate masses and inertias

File: gbeam_sim/gbeam_def.sdf.xacro (robot description, xacro)
@@ -9,9 +9,9 @@
       <pose>${pose}</pose>
       <inertial>
-        <mass>0.3</mass>
+        <mass>0.2</mass>
         <inertia>
-          <ixx>0.001</ixx><ixy>0</ixy>    <ixz>0</ixz>
-          <iyy>0.002</iyy><iyz>0</iyz>
-          <izz>0.001</izz>
+          <ixx>0.0001</ixx><ixy>0</ixy>    <ixz>0</ixz>
+          <iyy>0.0002</iyy><iyz>0</iyz>
+          <izz>0.0001</izz>
         </inertia>
       </inertial>
@@ -146,9 +146,9 @@
       <pose>${pose}</pose>
       <inertial>
-        <mass>0.2</mass>
+        <mass>0.1</mass>
         <inertia>
-          <ixx>0.001</ixx><ixy>0</ixy>    <ixz>0</ixz>
-          <iyy>0.001</iyy><iyz>0</iyz>
-          <izz>0.001</izz>
+          <ixx>5.22E-5</ixx><ixy>0</ixy>    <ixz>0</ixz>
+          <iyy>5.22E-5</iyy><iyz>0</iyz>
+          <izz>5.22E-5</izz>
         </inertia>
       </inertial>
@@ -253,8 +253,8 @@
               <cfm_damping>true</cfm_damping>
               <cfm>0.01</cfm>
-              <erp>0.05</erp>
+              <erp>0.03</erp>
               <limit>
                 <cfm>0.05</cfm>
-                <erp>0.05</erp>
+                <erp>0.03</erp>
               </limit>
             </ode>
