Commit message: adding re-mating and making mates closer

File: gbeam_sim/gbeam_def.sdf.xacro (robot description, xacro)
@@ -3,8 +3,31 @@
   <xacro:property name="pi" value="3.14159265"/>
   <!-- GBeam links -->
-  <xacro:macro name="gbeam_link" params="suffix pose">
-    <link name="gbeam_link${suffix}">
-      <gravity>1</gravity>
-      <self_collide>1</self_collide>
+  <xacro:macro name="gbeam_link" params="prefix suffix pose fixed">
+    <xacro:if value="${fixed}">
+      <joint name="${prefix}gbeam_link${suffix}_anchor" type="revolute">
+        <pose>0 0 0 0 0 0</pose>
+        <parent>world</parent>
+        <child>${prefix}gbeam_link${suffix}</child>
+        <axis>
+          <xyz>0 0 1</xyz>
+          <limit>
+            <lower>0</lower>
+            <upper>0</upper>
+          </limit>
+          <dynamics>
+            <damping>0</damping>
+          </dynamics>
+        </axis>
+      </joint>
+    </xacro:if>
+    <link name="${prefix}gbeam_link${suffix}">
+      <xacro:if value="${fixed}">
+        <gravity>0</gravity>
+        <self_collide>0</self_collide>
+      </xacro:if>
+      <xacro:unless value="${fixed}">
+        <gravity>1</gravity>
+        <self_collide>1</self_collide>
+      </xacro:unless>
       <pose>${pose}</pose>
       <inertial>
@@ -140,8 +163,31 @@
     </link>
   </xacro:macro>
-  <xacro:macro name="gbeam_node" params="suffix pose">
-    <link name="gbeam_node${suffix}">
-      <gravity>1</gravity>
-      <self_collide>1</self_collide>
+  <xacro:macro name="gbeam_node" params="prefix suffix pose fixed">
+    <xacro:if value="${fixed}">
+      <joint name="${prefix}gbeam_node${suffix}_anchor" type="revolute">
+        <pose>0 0 0 0 0 0</pose>
+        <parent>world</parent>
+        <child>${prefix}gbeam_node${suffix}</child>
+        <axis>
+          <xyz>0 0 1</xyz>
+          <limit>
+            <lower>0</lower>
+            <upper>0</upper>
+          </limit>
+          <dynamics>
+            <damping>0</damping>
+          </dynamics>
+        </axis>
+      </joint>
+    </xacro:if>
+    <link name="${prefix}gbeam_node${suffix}">
+      <xacro:if value="${fixed}">
+        <gravity>0</gravity>
+        <self_collide>0</self_collide>
+      </xacro:if>
+      <xacro:unless value="${fixed}">
+        <gravity>1</gravity>
+        <self_collide>1</self_collide>
+      </xacro:unless>
       <pose>${pose}</pose>
       <inertial>
@@ -203,10 +249,10 @@
       <collision name ='collision'>
         <geometry>
-          <sphere><radius>0.025</radius></sphere>
+          <sphere><radius>0.028</radius></sphere>
         </geometry>
       </collision>
       <visual name ='visual'>
         <geometry>
-          <sphere><radius>0.025</radius></sphere>
+          <sphere><radius>0.028</radius></sphere>
         </geometry>
       </visual>
@@ -239,5 +285,5 @@
         </detach_threshold>
         <joint type="prismatic" name="gbeam">
-          <pose>0 0.025 0 0 ${pi/2} 0</pose>
+          <pose>0 0.028 0 0 ${pi/2} 0</pose>
           <parent>gbeam_link</parent>
           <child>gbeam_node</child>
@@ -248,4 +294,7 @@
               <upper>0.001</upper>
             </limit>
+            <dynamics>
+              <damping>0.1</damping>
+            </dynamics>
           </axis>
           <physics>
@@ -253,8 +302,8 @@
               <cfm_damping>true</cfm_damping>
               <cfm>0.01</cfm>
-              <erp>0.03</erp>
+              <erp>0.02</erp>
               <limit>
-                <cfm>0.05</cfm>
-                <erp>0.03</erp>
+                <cfm>0.01</cfm>
+                <erp>0.01</erp>
               </limit>
             </ode>
@@ -267,8 +316,8 @@
     <atom_model type="gbeam_link">
       <mate_point type="gbeam" gender="male">
-        <pose>0 0.126 0 ${pi/2} ${pi/4} ${pi}</pose>
-      </mate_point>
-      <mate_point type="gbeam" gender="male">
-        <pose>0 -0.126 0 ${pi/2} ${pi/4} 0</pose>
+        <pose>0 0.122 0 ${pi/2} ${pi/4} ${pi}</pose>
+      </mate_point>
+      <mate_point type="gbeam" gender="male">
+        <pose>0 -0.122 0 ${pi/2} ${pi/4} 0</pose>
       </mate_point>
     </atom_model>
@@ -277,20 +326,20 @@
     <atom_model type="gbeam_node">
       <mate_point type="gbeam" gender="female">
-        <pose>0 0.025 0 ${pi/2} 0 0</pose>
-      </mate_point>
-      <mate_point type="gbeam" gender="female">
-        <pose>0 -0.025 0 ${pi/2} 0 ${pi}</pose>
-      </mate_point>
-      <mate_point type="gbeam" gender="female">
-        <pose>0 0 0.025 ${pi} 0 0</pose>
-      </mate_point>
-      <mate_point type="gbeam" gender="female">
-        <pose>0 0 -0.025 0 0 0</pose>
-      </mate_point>
-      <mate_point type="gbeam" gender="female">
-        <pose>0.025 0 0 0 -${pi/2.0} 0</pose>
-      </mate_point>
-      <mate_point type="gbeam" gender="female">
-        <pose>-0.025 0 0 0 ${pi/2.0} 0</pose>
+        <pose>0 0.028 0 ${pi/2} 0 0</pose>
+      </mate_point>
+      <mate_point type="gbeam" gender="female">
+        <pose>0 -0.028 0 ${pi/2} 0 ${pi}</pose>
+      </mate_point>
+      <mate_point type="gbeam" gender="female">
+        <pose>0 0 0.028 ${pi} 0 0</pose>
+      </mate_point>
+      <mate_point type="gbeam" gender="female">
+        <pose>0 0 -0.028 0 0 0</pose>
+      </mate_point>
+      <mate_point type="gbeam" gender="female">
+        <pose>0.028 0 0 0 -${pi/2.0} 0</pose>
+      </mate_point>
+      <mate_point type="gbeam" gender="female">
+        <pose>-0.028 0 0 0 ${pi/2.0} 0</pose>
       </mate_point>
     </atom_model>
@@ -299,38 +348,38 @@
     <atom_model type="hog">
       <mate_point type="gbeam" gender="female">
-        <pose>0 0.025 0 ${pi/2} 0 0</pose>
-      </mate_point>
-      <mate_point type="gbeam" gender="female">
-        <pose>0 -0.025 0 ${pi/2} 0 ${pi}</pose>
-      </mate_point>
-      <mate_point type="gbeam" gender="female">
-        <pose>0 0 0.025 ${pi} 0 0</pose>
-      </mate_point>
-      <mate_point type="gbeam" gender="female">
-        <pose>0 0 -0.025 0 0 0</pose>
-      </mate_point>
-      <mate_point type="gbeam" gender="female">
-        <pose>0.025 0 0 0 -${pi/2.0} 0</pose>
-      </mate_point>
-      <mate_point type="gbeam" gender="female">
-        <pose>-0.025 0 0 0 ${pi/2.0} 0</pose>
-      </mate_point>
-      <mate_point type="gbeam" gender="male">
-        <pose>0 -0.025 0 ${pi/2} 0 0</pose>
-      </mate_point>
-      <mate_point type="gbeam" gender="male">
-        <pose>0 0.025 0 ${pi/2} 0 ${pi}</pose>
-      </mate_point>
-      <mate_point type="gbeam" gender="male">
-        <pose>0 0 -0.025 ${pi} 0 0</pose>
-      </mate_point>
-      <mate_point type="gbeam" gender="male">
-        <pose>0 0 0.025 0 0 0</pose>
-      </mate_point>
-      <mate_point type="gbeam" gender="male">
-        <pose>-0.025 0 0 0 -${pi/2.0} 0</pose>
-      </mate_point>
-      <mate_point type="gbeam" gender="male">
-        <pose>0.025 0 0 0 ${pi/2.0} 0</pose>
+        <pose>0 0.028 0 ${pi/2} 0 0</pose>
+      </mate_point>
+      <mate_point type="gbeam" gender="female">
+        <pose>0 -0.028 0 ${pi/2} 0 ${pi}</pose>
+      </mate_point>
+      <mate_point type="gbeam" gender="female">
+        <pose>0 0 0.028 ${pi} 0 0</pose>
+      </mate_point>
+      <mate_point type="gbeam" gender="female">
+        <pose>0 0 -0.028 0 0 0</pose>
+      </mate_point>
+      <mate_point type="gbeam" gender="female">
+        <pose>0.028 0 0 0 -${pi/2.0} 0</pose>
+      </mate_point>
+      <mate_point type="gbeam" gender="female">
+        <pose>-0.028 0 0 0 ${pi/2.0} 0</pose>
+      </mate_point>
+      <mate_point type="gbeam" gender="male">
+        <pose>0 -0.028 0 ${pi/2} 0 0</pose>
+      </mate_point>
+      <mate_point type="gbeam" gender="male">
+        <pose>0 0.028 0 ${pi/2} 0 ${pi}</pose>
+      </mate_point>
+      <mate_point type="gbeam" gender="male">
+        <pose>0 0 -0.028 ${pi} 0 0</pose>
+      </mate_point>
+      <mate_point type="gbeam" gender="male">
+        <pose>0 0 0.028 0 0 0</pose>
+      </mate_point>
+      <mate_point type="gbeam" gender="male">
+        <pose>-0.028 0 0 0 -${pi/2.0} 0</pose>
+      </mate_point>
+      <mate_point type="gbeam" gender="male">
+        <pose>0.028 0 0 0 ${pi/2.0} 0</pose>
       </mate_point>
     </atom_model>

Commit message: changing dipole sim to use hard joint constraints

File: gbeam_sim/gbeam_def.sdf.xacro (robot description, xacro)
@@ -241,6 +241,6 @@
       <frameId>hog</frameId>
       <linkName>hog</linkName>
-      <kl>400</kl>
-      <ka>200</ka>
+      <kl>100</kl>
+      <ka>50</ka>
     </plugin>
     <link name ='hog'>
@@ -286,23 +286,25 @@
         <!-- four-magnet mate -->
         <xacro:if value="1">
+          <max_force>50.0 50.0 10.0</max_force>
+          <max_torque>0.5 0.5 5.0</max_torque>
           <dipole>
             <position>0.01 0.01 0</position>
-            <moment>0 0 0.08</moment>
-            <min_distance>0.004</min_distance>
+            <moment>0 0 0.02</moment>
+            <min_distance>0.003</min_distance>
           </dipole>
           <dipole>
             <position>-0.1 0.01 0</position>
-            <moment>0 0 0.08</moment>
-            <min_distance>0.004</min_distance>
+            <moment>0 0 0.02</moment>
+            <min_distance>0.003</min_distance>
           </dipole>
           <dipole>
             <position>-0.01 -0.01 0</position>
-            <moment>0 0 0.08</moment>
-            <min_distance>0.004</min_distance>
+            <moment>0 0 0.02</moment>
+            <min_distance>0.003</min_distance>
           </dipole>
           <dipole>
             <position>0.01 -0.01 0</position>
-            <moment>0 0 0.08</moment>
-            <min_distance>0.004</min_distance>
+            <moment>0 0 0.02</moment>
+            <min_distance>0.003</min_distance>
           </dipole>
         </xacro:if>
@@ -335,12 +337,13 @@
           </axis>
           <physics>
+            <provide_feedback>true</provide_feedback>
             <ode>
-              <cfm_damping>true</cfm_damping>
-              <cfm>0.001</cfm>
-              <erp>0.02</erp>
-              <limit>
-                <cfm>0.001</cfm>
-                <erp>0.01</erp>
-              </limit>
+              <!--<cfm_damping>true</cfm_damping>-->
+              <!--<cfm>1.0</cfm>-->
+              <!--<erp>0.02</erp>-->
+              <!--<limit>-->
+                <!--<cfm>0.001</cfm>-->
+                <!--<erp>0.01</erp>-->
+              <!--</limit>-->
             </ode>
           </physics>

File: gbeam_sim/gbeam_soup.sdf.xacro (robot description, xacro)
@@ -23,13 +23,16 @@
     <!-- Create the initial scene made of links and nodes -->
     <xacro:gbeam_node fixed="false" prefix="" suffix="_1" pose="0 0.3 0.1 0 0 0"/>
-    <!--<xacro:gbeam_node fixed="false" prefix="" suffix="_2" pose="0 0.3 0.2 0 0 0"/>-->
-    <!--<xacro:gbeam_node fixed="false" prefix="" suffix="_3" pose="0 0.3 0.3 0 0 0"/>-->
-    <xacro:gbeam_node fixed="false" prefix="" suffix="_2" pose="0.0 -0.280 0.1 0 0 0"/>
+    <xacro:gbeam_node fixed="false" prefix="" suffix="_2" pose="0 0.3 0.2 0 0 0"/>
+    <xacro:gbeam_node fixed="false" prefix="" suffix="_3" pose="0 0.3 0.3 0 0 0"/>
+    <!--<xacro:gbeam_node fixed="false" prefix="" suffix="_4" pose="0.0 -0.280 0.1 0 0 0"/>-->
     <!--<xacro:gbeam_node fixed="false" prefix="" suffix="_3" pose="0.0 -0.520 0.1 0 0 0"/>-->
     <!--<xacro:gbeam_node fixed="false" prefix="" suffix="_4" pose="0.0 -0.2 0.1 0 0 0"/>-->
     <!--<xacro:gbeam_node suffix="_4" pose="0 0 0.3 0 0 0"/>-->
     <!--<xacro:gbeam_node suffix="_5" pose="0 0 0.4 0 0 0"/>-->
-    <xacro:gbeam_link fixed="false" prefix="" suffix="_1" pose="0 -0.5 0.4 0 0.785398163 0"/>
-    <xacro:gbeam_link fixed="false" prefix="" suffix="_2" pose="0.0 0.0 0.26 1.5707 0 0"/>
+    <xacro:gbeam_link fixed="false" prefix="" suffix="_1" pose="0.0 0.0 0.26 1.5707 0 0.785398163"/>
+    <xacro:gbeam_link fixed="false" prefix="" suffix="_2" pose="0 0.8 0.2 0 0.785398163 0"/>
+    <xacro:gbeam_link fixed="false" prefix="" suffix="_3" pose="0 0.8 0.3 0 0.785398163 0"/>
+    <xacro:gbeam_link fixed="false" prefix="" suffix="_4" pose="0 0.8 0.4 0 0.785398163 0"/>
+    <xacro:gbeam_link fixed="false" prefix="" suffix="_5" pose="0 0.8 0.5 0 0.785398163 0"/>
     <!--<xacro:gbeam_link suffix="_3" pose="0 0.1 0.2 0 0 0"/>-->
     <!--<xacro:gbeam_link suffix="_4" pose="0 0.1 0.3 0 0 0"/>-->

Commit message: fixing bad magnet model in gbeam_def adding a ton of introspection

File: gbeam_sim/gbeam_def.sdf.xacro (robot description, xacro)
@@ -77,5 +77,5 @@
             <friction>
               <ode>
-                <mu>0.7</mu>
+                <mu>0.2</mu>
                 <!--<mu2>0.7</mu2>-->
               </ode>
@@ -207,5 +207,5 @@
           <friction>
             <ode>
-              <mu>0.5</mu>
+              <mu>0.2</mu>
               <!--<mu2>0.5</mu2>-->
             </ode>
@@ -268,5 +268,5 @@
   </xacro:macro>
   <!-- GBeam mates -->
-  <xacro:macro name="gbeam_mate" params="linear_attach angular_attach linear_detach angular_detach">
+  <xacro:macro name="gbeam_mate">
     <mate_model type="gbeam" model="dipole">
       <!-- planar shear-supporting magnetic mate
@@ -286,6 +286,7 @@
         <!-- four-magnet mate -->
         <xacro:if value="1">
-          <max_force>50.0 50.0 10.0</max_force>
-          <max_torque>0.5 0.5 5.0</max_torque>
+          <max_force>70.0 70.0 15.0</max_force>
+          <max_torque>1.5 1.5 9.0</max_torque>
+          <max_distance>0.03</max_distance>
           <dipole>
             <position>0.01 0.01 0</position>
@@ -294,5 +295,5 @@
           </dipole>
           <dipole>
-            <position>-0.1 0.01 0</position>
+            <position>-0.01 0.01 0</position>
             <moment>0 0 0.02</moment>
             <min_distance>0.003</min_distance>
@@ -311,29 +312,27 @@
         <!-- proximity -->
         <attach_threshold>
-          <linear>0.0005</linear>
+          <linear>0.005</linear>
           <angular>0.05</angular>
-          <!--<linear>${linear_attach}</linear>-->
-          <!--<angular>${angular_attach}</angular>-->
         </attach_threshold>
         <detach_threshold>
-          <linear>0.005</linear>
-          <angular>0.05</angular>
-          <!--<linear>${linear_detach}</linear>-->
-          <!--<angular>${angular_detach}</angular>-->
+          <linear>0.015</linear>
+          <angular>0.15</angular>
         </detach_threshold>
-        <joint type="prismatic" name="gbeam">
+        <joint type="fixed" name="gbeam">
           <pose>0 0.028 0 0 ${pi/2} 0</pose>
           <parent>gbeam_link</parent>
           <child>gbeam_node</child>
-          <axis>
-            <xyz>0 0 1</xyz>
-            <limit>
-              <lower>-0.0001</lower>
-              <upper>0.0001</upper>
-            </limit>
-            <dynamics>
-              <damping>0.1</damping>
-            </dynamics>
-          </axis>
+          <xacro:if value="0">
+            <axis>
+              <xyz>0 0 1</xyz>
+              <limit>
+                <lower>-0.0001</lower>
+                <upper>0.0001</upper>
+              </limit>
+              <dynamics>
+                <damping>0.1</damping>
+              </dynamics>
+            </axis>
+          </xacro:if>
           <physics>
             <provide_feedback>true</provide_feedback>

File: gbeam_sim/gbeam_soup.sdf.xacro (robot description, xacro)
@@ -9,9 +9,5 @@
       <publish_active_mates>1</publish_active_mates>
       <!-- Mate Models -->
-      <xacro:gbeam_mate
-        linear_attach="0.025"
-        linear_detach="0.030"
-        angular_attach="0.15"
-        angular_detach="0.20"/>
+      <xacro:gbeam_mate/>
       <!-- Atom Models -->
       <xacro:gbeam_link_atom/>

Commit message: improving visualization and simulation accuracy

File: gbeam_sim/gbeam_def.sdf.xacro (robot description, xacro)
@@ -49,5 +49,5 @@
               <ode>
                 <mu>0.7</mu>
-                <!--<mu2>0.7</mu2>-->
+                <!--<mu2>0.1</mu2>-->
               </ode>
             </friction>
@@ -57,8 +57,8 @@
             <contact>
               <ode>
-                <soft_cfm>0.01</soft_cfm>
-                <soft_erp>0.05</soft_erp>
-                <kp>50000</kp>
-                <kd>8</kd>
+                <!--<soft_cfm>0.01</soft_cfm>-->
+                <!--<soft_erp>0.05</soft_erp>-->
+                <!--<kp>50000</kp>-->
+                <!--<kd>8</kd>-->
               </ode>
             </contact>
@@ -67,4 +67,5 @@
       </xacro:unless>
       <xacro:if value="true">
+        <!-- Beam -->
         <collision name='gbeam_link_collision'>
           <pose>0 0 0 0 -0 0</pose>
@@ -88,10 +89,11 @@
                 <soft_cfm>0.01</soft_cfm>
                 <soft_erp>0.05</soft_erp>
-                <kp>50000</kp>
-                <kd>8</kd>
+                <!--<kp>5000</kp>-->
+                <!--<kd>0.2</kd>-->
               </ode>
             </contact>
           </surface>
         </collision>
+        <!-- Top Cap -->
         <collision name='gbeam_link_collision_gbeam_link_1'>
           <pose>0 ${0.115-0.00635/2.0} 0 1.5707 -0 0</pose>
@@ -105,5 +107,5 @@
             <friction>
               <ode>
-                <mu>1.7</mu>
+                <mu>0.9</mu>
                 <!--<mu2>0.7</mu2>-->
                 <slip1>1.0</slip1>
@@ -119,4 +121,5 @@
           </surface>
         </collision>
+        <!-- Bottom Cap -->
         <collision name='gbeam_link_collision_gbeam_link_2'>
           <pose>0 ${-0.115+0.00635/2.0} 0 1.5707 -0 0</pose>
@@ -130,5 +133,5 @@
             <friction>
               <ode>
-                <mu>1.7</mu>
+                <mu>0.9</mu>
                 <slip1>1.0</slip1>
                 <slip2>1.0</slip2>
@@ -143,6 +146,4 @@
                 <soft_cfm>0.01</soft_cfm>
                 <soft_erp>0.02</soft_erp>
-                <kp>50000</kp>
-                <kd>8</kd>
               </ode>
             </contact>
@@ -150,10 +151,10 @@
         </collision>
       </xacro:if>
-      <visual name='visual'>
+      <visual name='gbeam_link_visual'>
         <material>
-          <ambient>0.6 0.6 0.6 1</ambient>
-          <diffuse>0.5 0.5 0.5 1</diffuse>
-          <specular>1.0 1.0 1.0 1</specular>
-          <emissive>0 0 0 0</emissive>
+          <script>
+            <uri>file://$(find gbeam_model)/urdf/gbeam.material</uri>
+            <name>Gbeam/Link</name>
+          </script>
         </material>
         <geometry>
@@ -207,5 +208,5 @@
           <friction>
             <ode>
-              <mu>0.2</mu>
+              <mu>0.8</mu>
               <!--<mu2>0.5</mu2>-->
             </ode>
@@ -219,15 +220,15 @@
               <soft_erp>0.02</soft_erp>
               <kp>50000</kp>
-              <kd>8</kd>
+              <kd>0.2</kd>
             </ode>
           </contact>
         </surface>
       </collision>
-      <visual name='visual'>
+      <visual name='gbeam_node_visual'>
         <material>
-          <ambient>0.3 0.3 0.3 1</ambient>
-          <diffuse>0.5 0.5 0.5 1</diffuse>
-          <specular>1.0 1.0 1.0 1</specular>
-          <emissive>0 0 0 0</emissive>
+          <script>
+            <uri>file://$(find gbeam_model)/urdf/gbeam.material</uri>
+            <name>Gbeam/Node</name>
+          </script>
         </material>
         <geometry>
@@ -286,25 +287,29 @@
         <!-- four-magnet mate -->
         <xacro:if value="1">
-          <max_force>70.0 70.0 15.0</max_force>
-          <max_torque>1.5 1.5 9.0</max_torque>
+          <!-- This is the maximum force in the mate frame before the mate detaches -->
+          <max_force>70.0 70.0 10.0</max_force>
+          <!-- This is the maximum torque in the mate frame before the mate detaches -->
+          <max_torque>1.7 1.7 9.0</max_torque>
+          <!-- This is the maximum distance between the mate points before the mate detaches -->
           <max_distance>0.03</max_distance>
+          <!-- Four diples arranged in a cross patter, aligned pointing out along the local z axis -->
           <dipole>
             <position>0.01 0.01 0</position>
-            <moment>0 0 0.02</moment>
+            <moment>0 0 0.03</moment>
             <min_distance>0.003</min_distance>
           </dipole>
           <dipole>
             <position>-0.01 0.01 0</position>
-            <moment>0 0 0.02</moment>
+            <moment>0 0 0.03</moment>
             <min_distance>0.003</min_distance>
           </dipole>
           <dipole>
             <position>-0.01 -0.01 0</position>
-            <moment>0 0 0.02</moment>
+            <moment>0 0 0.03</moment>
             <min_distance>0.003</min_distance>
           </dipole>
           <dipole>
             <position>0.01 -0.01 0</position>
-            <moment>0 0 0.02</moment>
+            <moment>0 0 0.03</moment>
             <min_distance>0.003</min_distance>
           </dipole>
@@ -312,6 +317,6 @@
         <!-- proximity -->
         <attach_threshold>
-          <linear>0.0005</linear>
-          <angular>0.005</angular>
+          <linear>0.001</linear>
+          <angular>0.01</angular>
         </attach_threshold>
         <detach_threshold>
